File: _autosave-amps.sch (KiCad schematic (older format))
At the start: 5 parts

Commit message: Amplifier
Added initial amplifier file amps.sch
Connections:
- net labels added: EN
Changed lines of the file:
@@
 EESchema Schematic File Version 4
+LIBS:daq-hardware-cache
 EELAYER 30 0
 EELAYER END
 $Descr A4 11693 8268
 encoding utf-8
-Sheet 1 1
+Sheet 2 3
 Title ""
 Date ""
@@
 Wire Wire Line
 	4100 3500 4100 3650
+Text HLabel 6850 3350 2    50   Input ~ 0
+EN
 $EndSCHEMATC
