File: amps.sch (KiCad schematic (older format))
At the start: 0 parts

Commit message: Amplifier
Parts:
- added C?: C, symbol Device:C
- added J?: Screw_Terminal_01x04, symbol Connector:Screw_Terminal_01x04
- added R? (x2): R, symbol Device:R
- added U?: MCP6N11, symbol RMTS-cache:RMTS-rescue_MCP6N11-Mine-RMTS-rescue-RMTS-rescue
Connections:
- net labels added: EN, GND
- wire segments 0 -> 27
Changed lines of the file:
@@
 EESchema Schematic File Version 4
-EELAYER 29 0
+LIBS:daq-hardware-cache
+EELAYER 30 0
 EELAYER END
 $Descr A4 11693 8268
 encoding utf-8
-Sheet 1 3
+Sheet 2 3
 Title ""
 Date ""
@@
 Comment4 ""
 $EndDescr
+$Comp
+L RMTS-cache:RMTS-rescue_MCP6N11-Mine-RMTS-rescue-RMTS-rescue U?
+U 1 1 5DAB7967
+P 5950 3350
+F 0 "U?" H 5950 3575 50  0000 C CNN
+F 1 "MCP6N11" H 5950 3484 50  0000 C CNN
+F 2 "" H 5950 3350 50  0001 C CNN
+F 3 "" H 5950 3350 50  0001 C CNN
+	1    5950 3350
+	1    0    0    -1
+$EndComp
+$Comp
+L Connector:Screw_Terminal_01x04 J?
+U 1 1 5DAB817A
+P 3700 3500
+F 0 "J?" H 3618 3075 50  0000 C CNN
+F 1 "Screw_Terminal_01x04" H 3618 3166 50  0000 C CNN
+F 2 "" H 3700 3500 50  0001 C CNN
+F 3 "~" H 3700 3500 50  0001 C CNN
+	1    3700 3500
+	-1   0    0    1
+$EndComp
+$Comp
+L power:GND #PWR?
+U 1 1 5DABC36F
+P 5400 4200
+F 0 "#PWR?" H 5400 3950 50  0001 C CNN
+F 1 "GND" H 5405 4027 50  0000 C CNN
+F 2 "" H 5400 4200 50  0001 C CNN
+F 3 "" H 5400 4200 50  0001 C CNN
+	1    5400 4200
+	1    0    0    -1
+$EndComp
+$Comp
+L power:GND #PWR?
+U 1 1 5DABC657
+P 5400 4200
+F 0 "#PWR?" H 5400 3950 50  0001 C CNN
+F 1 "GND" H 5405 4027 50  0000 C CNN
+F 2 "" H 5400 4200 50  0001 C CNN
+F 3 "" H 5400 4200 50  0001 C CNN
+	1    5400 4200
+	1    0    0    -1
+$EndComp
+Wire Wire Line
+	5400 4200 5400 3650
+Wire Wire Line
+	5400 3650 5550 3650
+$Comp
+L Device:R R?
+U 1 1 5DABEACC
+P 6550 3900
+F 0 "R?" H 6620 3946 50  0000 L CNN
+F 1 "R" H 6620 3855 50  0000 L CNN
+F 2 "" V 6480 3900 50  0001 C CNN
+F 3 "~" H 6550 3900 50  0001 C CNN
+	1    6550 3900
+	1    0    0    -1
+$EndComp
+Wire Wire Line
+	6550 3650 6550 3750
+Wire Wire Line
+	6550 3650 6850 3650
+$Comp
+L Device:R R?
+U 1 1 5DABF163
+P 6550 4400
+F 0 "R?" H 6620 4446 50  0000 L CNN
+F 1 "R" H 6620 4355 50  0000 L CNN
+F 2 "" V 6480 4400 50  0001 C CNN
+F 3 "~" H 6550 4400 50  0001 C CNN
+	1    6550 4400
+	1    0    0    -1
+$EndComp
+Wire Wire Line
+	6550 4050 6550 4150
+Wire Wire Line
+	6550 4150 6850 4150
+Connection ~ 6550 4150
+Wire Wire Line
+	6550 4150 6550 4250
+$Comp
+L power:GND #PWR?
+U 1 1 5DABFAE9
+P 6350 4600
+F 0 "#PWR?" H 6350 4350 50  0001 C CNN
+F 1 "GND" H 6355 4427 50  0000 C CNN
+F 2 "" H 6350 4600 50  0001 C CNN
+F 3 "" H 6350 4600 50  0001 C CNN
+	1    6350 4600
+	1    0    0    -1
+$EndComp
+Wire Wire Line
+	6350 3650 6350 4600
+Wire Wire Line
+	6550 4550 6550 4600
+Wire Wire Line
+	6550 4600 6350 4600
+Connection ~ 6350 4600
+Wire Wire Line
+	6350 3550 6550 3550
+Wire Wire Line
+	6550 3550 6550 3650
+Connection ~ 6550 3650
+Wire Wire Line
+	6350 3450 6850 3450
+Wire Wire Line
+	6350 3350 6850 3350
+$Comp
+L Device:C C?
+U 1 1 5DAC169D
+P 4700 3450
+F 0 "C?" H 4815 3496 50  0000 L CNN
+F 1 "C" H 4815 3405 50  0000 L CNN
+F 2 "" H 4738 3300 50  0001 C CNN
+F 3 "~" H 4700 3450 50  0001 C CNN
+	1    4700 3450
+	1    0    0    -1
+$EndComp
+Wire Wire Line
+	3900 3400 4350 3400
+Wire Wire Line
+	4350 3400 4350 3600
+Wire Wire Line
+	4350 3600 4700 3600
+Wire Wire Line
+	3900 3300 4700 3300
+Wire Wire Line
+	4700 3300 5150 3300
+Wire Wire Line
+	5150 3300 5150 3450
+Wire Wire Line
+	5150 3450 5550 3450
+Connection ~ 4700 3300
+Wire Wire Line
+	4700 3600 5550 3600
+Wire Wire Line
+	5550 3600 5550 3550
+Connection ~ 4700 3600
+Wire Wire Line
+	5550 3350 5300 3350
+$Comp
+L power:GND #PWR?
+U 1 1 5DAC322E
+P 3900 3800
+F 0 "#PWR?" H 3900 3550 50  0001 C CNN
+F 1 "GND" H 3905 3627 50  0000 C CNN
+F 2 "" H 3900 3800 50  0001 C CNN
+F 3 "" H 3900 3800 50  0001 C CNN
+	1    3900 3800
+	1    0    0    -1
+$EndComp
+Wire Wire Line
+	3900 3600 3900 3800
+Wire Wire Line
+	3900 3500 4100 3500
+Wire Wire Line
+	4100 3500 4100 3650
+Text HLabel 6850 3350 2    50   Input ~ 0
+EN
 $EndSCHEMATC
