File: _autosave-daq-hardware.sch (KiCad schematic (older format))
At the start: 9 parts, among them J1 USB_B, J2 Micro_SD_Card_Det_Hirose_DM3AT, Q1 MMDT2222A, U1 CP2102N-A01-GQFN24, U2 ESP32-WROOM-32D

Commit message: amplifier changes
Changed lines of the file:
@@
 GPIO0
 $Sheet
-S 8250 4450 1200 550
+S 8250 4300 1200 550
 U 5DAADE1C
 F0 "amps" 50
 F1 "amps.sch" 50
-F2 "EN" I L 8250 4550 50
+F2 "EN" I L 8250 4400 50
 $EndSheet
 $Sheet
