File: thermocouples.sch (KiCad schematic (older format))
At the start: 16 parts

Commit message: Thermocouples
Added components to the PCB. Please check the GND and VCC lines arrangement for any changes.
Parts:
- gave numbers to parts that had none: 16
Connections:
- net T1_T+: now also J3.2 (Pin_2); no longer J3.1 (Pin_1)
- net T1_T-: now also J3.1 (Pin_1); no longer J3.2 (Pin_2)
- net T2_T+: now also J4.2 (Pin_2); no longer J4.1 (Pin_1)
- net T2_T-: now also J4.1 (Pin_1); no longer J4.2 (Pin_2)
- net T3_T+: now also J5.2 (Pin_2); no longer J5.1 (Pin_1)
- net T3_T-: now also J5.1 (Pin_1); no longer J5.2 (Pin_2)
- net T4_T+: now also J6.2 (Pin_2); no longer J6.1 (Pin_1)
- net T4_T-: now also J6.1 (Pin_1); no longer J6.2 (Pin_2)
Changed lines of the file:
@@
 $EndDescr
 $Comp
-L Sensor_Temperature:MAX31855RASA U?
+L Sensor_Temperature:MAX31855RASA U4
 U 1 1 5DA6096E
 P 2950 2400
-F 0 "U?" H 2950 2981 50  0000 C CNN
+F 0 "U4" H 2950 2981 50  0000 C CNN
 F 1 "MAX31855RASA" H 2950 2890 50  0000 C CNN
 F 2 "Package_SO:SOIC-8_3.9x4.9mm_P1.27mm" H 3950 2050 50  0001 C CIN
@@
 $EndComp
 $Comp
-L Device:C C?
+L Device:C C4
 U 1 1 5DA633EE
 P 2000 2400
-F 0 "C?" H 2115 2446 50  0000 L CNN
+F 0 "C4" H 2115 2446 50  0000 L CNN
 F 1 "100nF" H 2115 2355 50  0000 L CNN
 F 2 "Capacitor_SMD:C_0603_1608Metric" H 2038 2250 50  0001 C CNN
@@
 	2000 2000 2000 2250
 $Comp
-L power:+3V3 #PWR?
+L power:+3V3 #PWR0117
 U 1 1 5DA64666
 P 2000 1900
-F 0 "#PWR?" H 2000 1750 50  0001 C CNN
+F 0 "#PWR0117" H 2000 1750 50  0001 C CNN
 F 1 "+3V3" H 2015 2073 50  0000 C CNN
 F 2 "" H 2000 1900 50  0001 C CNN
@@
 Connection ~ 2000 2000
 $Comp
-L power:GND #PWR?
+L power:GND #PWR0118
 U 1 1 5DA65041
 P 2000 2900
-F 0 "#PWR?" H 2000 2650 50  0001 C CNN
+F 0 "#PWR0118" H 2000 2650 50  0001 C CNN
 F 1 "GND" H 2005 2727 50  0000 C CNN
 F 2 "" H 2000 2900 50  0001 C CNN
@@
 Connection ~ 2000 2800
 $Comp
-L Device:C C?
+L Device:C C5
 U 1 1 5DA6662C
 P 2400 2400
-F 0 "C?" H 2515 2446 50  0000 L CNN
+F 0 "C5" H 2515 2446 50  0000 L CNN
 F 1 "10nF" H 2515 2355 50  0000 L CNN
 F 2 "Capacitor_SMD:C_0603_1608Metric" H 2438 2250 50  0001 C CNN
@@
 	2550 2550 2400 2550
 $Comp
-L Sensor_Temperature:MAX31855RASA U?
+L Sensor_Temperature:MAX31855RASA U6
 U 1 1 5DAB048A
 P 6950 2400
-F 0 "U?" H 6950 2981 50  0000 C CNN
+F 0 "U6" H 6950 2981 50  0000 C CNN
 F 1 "MAX31855RASA" H 6950 2890 50  0000 C CNN
 F 2 "Package_SO:SOIC-8_3.9x4.9mm_P1.27mm" H 7950 2050 50  0001 C CIN
@@
 $EndComp
 $Comp
-L Device:C C?
+L Device:C C8
 U 1 1 5DAB0490
 P 6000 2400
-F 0 "C?" H 6115 2446 50  0000 L CNN
+F 0 "C8" H 6115 2446 50  0000 L CNN
 F 1 "100nF" H 6115 2355 50  0000 L CNN
 F 2 "Capacitor_SMD:C_0603_1608Metric" H 6038 2250 50  0001 C CNN
@@
 	6000 2000 6000 2250
 $Comp
-L power:+3V3 #PWR?
+L power:+3V3 #PWR0119
 U 1 1 5DAB049A
 P 6000 1900
-F 0 "#PWR?" H 6000 1750 50  0001 C CNN
+F 0 "#PWR0119" H 6000 1750 50  0001 C CNN
 F 1 "+3V3" H 6015 2073 50  0000 C CNN
 F 2 "" H 6000 1900 50  0001 C CNN
@@
 Connection ~ 6000 2000
 $Comp
-L power:GND #PWR?
+L power:GND #PWR0120
 U 1 1 5DAB04A2
 P 6000 2900
-F 0 "#PWR?" H 6000 2650 50  0001 C CNN
+F 0 "#PWR0120" H 6000 2650 50  0001 C CNN
 F 1 "GND" H 6005 2727 50  0000 C CNN
 F 2 "" H 6000 2900 50  0001 C CNN
@@
 Connection ~ 6000 2800
 $Comp
-L Device:C C?
+L Device:C C9
 U 1 1 5DAB04AA
 P 6400 2400
-F 0 "C?" H 6515 2446 50  0000 L CNN
+F 0 "C9" H 6515 2446 50  0000 L CNN
 F 1 "10nF" H 6515 2355 50  0000 L CNN
 F 2 "Capacitor_SMD:C_0603_1608Metric" H 6438 2250 50  0001 C CNN
@@
 	6550 2550 6400 2550
 $Comp
-L Device:C C?
+L Device:C C6
 U 1 1 5DAB1C47
 P 4000 2400
-F 0 "C?" H 4115 2446 50  0000 L CNN
+F 0 "C6" H 4115 2446 50  0000 L CNN
 F 1 "100nF" H 4115 2355 50  0000 L CNN
 F 2 "Capacitor_SMD:C_0603_1608Metric" H 4038 2250 50  0001 C CNN
@@
 	4000 2000 4000 2250
 $Comp
-L power:+3V3 #PWR?
+L power:+3V3 #PWR0121
 U 1 1 5DAB1C51
 P 4000 1900
-F 0 "#PWR?" H 4000 1750 50  0001 C CNN
+F 0 "#PWR0121" H 4000 1750 50  0001 C CNN
 F 1 "+3V3" H 4015 2073 50  0000 C CNN
 F 2 "" H 4000 1900 50  0001 C CNN
@@
 Connection ~ 4000 2000
 $Comp
-L power:GND #PWR?
+L power:GND #PWR0122
 U 1 1 5DAB1C59
 P 4000 2900
-F 0 "#PWR?" H 4000 2650 50  0001 C CNN
+F 0 "#PWR0122" H 4000 2650 50  0001 C CNN
 F 1 "GND" H 4005 2727 50  0000 C CNN
 F 2 "" H 4000 2900 50  0001 C CNN
@@
 Connection ~ 4000 2800
 $Comp
-L Device:C C?
+L Device:C C7
 U 1 1 5DAB1C61
 P 4400 2400
-F 0 "C?" H 4515 2446 50  0000 L CNN
+F 0 "C7" H 4515 2446 50  0000 L CNN
 F 1 "10nF" H 4515 2355 50  0000 L CNN
 F 2 "Capacitor_SMD:C_0603_1608Metric" H 4438 2250 50  0001 C CNN
@@
 	4550 2550 4400 2550
 $Comp
-L Sensor_Temperature:MAX31855RASA U?
+L Sensor_Temperature:MAX31855RASA U7
 U 1 1 5DAC2196
 P 8950 2400
-F 0 "U?" H 8950 2981 50  0000 C CNN
+F 0 "U7" H 8950 2981 50  0000 C CNN
 F 1 "MAX31855RASA" H 8950 2890 50  0000 C CNN
 F 2 "Package_SO:SOIC-8_3.9x4.9mm_P1.27mm" H 9950 2050 50  0001 C CIN
@@
 $EndComp
 $Comp
-L Device:C C?
+L Device:C C10
 U 1 1 5DAC219C
 P 8000 2400
-F 0 "C?" H 8115 2446 50  0000 L CNN
+F 0 "C10" H 8115 2446 50  0000 L CNN
 F 1 "100nF" H 8115 2355 50  0000 L CNN
 F 2 "Capacitor_SMD:C_0603_1608Metric" H 8038 2250 50  0001 C CNN
@@
 	8000 2000 8000 2250
 $Comp
-L power:+3V3 #PWR?
+L power:+3V3 #PWR0123
 U 1 1 5DAC21A6
 P 8000 1900
-F 0 "#PWR?" H 8000 1750 50  0001 C CNN
+F 0 "#PWR0123" H 8000 1750 50  0001 C CNN
 F 1 "+3V3" H 8015 2073 50  0000 C CNN
 F 2 "" H 8000 1900 50  0001 C CNN
@@
 Connection ~ 8000 2000
 $Comp
-L power:GND #PWR?
+L power:GND #PWR0124
 U 1 1 5DAC21AE
 P 8000 2900
-F 0 "#PWR?" H 8000 2650 50  0001 C CNN
+F 0 "#PWR0124" H 8000 2650 50  0001 C CNN
 F 1 "GND" H 8005 2727 50  0000 C CNN
 F 2 "" H 8000 2900 50  0001 C CNN
@@
 Connection ~ 8000 2800
 $Comp
-L Device:C C?
+L Device:C C11
 U 1 1 5DAC21B6
 P 8400 2400
-F 0 "C?" H 8515 2446 50  0000 L CNN
+F 0 "C11" H 8515 2446 50  0000 L CNN
 F 1 "10nF" H 8515 2355 50  0000 L CNN
 F 2 "Capacitor_SMD:C_0603_1608Metric" H 8438 2250 50  0001 C CNN
@@
 	2400 2250 2400 2100
 Connection ~ 2400 2250
-Text Label 2000 1500 0    50   ~ 0
+Text Label 2000 1600 0    50   ~ 0
 T1_T+
 Wire Wire Line
 	2400 2550 2400 2700
 Connection ~ 2400 2550
-Text Label 2000 1600 0    50   ~ 0
+Text Label 2000 1500 0    50   ~ 0
 T1_T-
 $Comp
-L Connector:Screw_Terminal_01x02 J?
+L Connector:Screw_Terminal_01x02 J3
 U 1 1 5DAD8258
 P 2550 1500
-F 0 "J?" H 2630 1492 50  0000 L CNN
+F 0 "J3" H 2630 1492 50  0000 L CNN
 F 1 "Screw_Terminal_Thermo_1" H 2630 1401 50  0000 L CNN
 F 2 "TerminalBlock_Phoenix:TerminalBlock_Phoenix_MPT-0,5-2-2.54_1x02_P2.54mm_Horizontal" H 2550 1500 50  0001 C CNN
@@
 T2_T-
 $Comp
-L Connector:Screw_Terminal_01x02 J?
+L Connector:Screw_Terminal_01x02 J4
 U 1 1 5DAE1281
 P 4550 1500
-F 0 "J?" H 4630 1492 50  0000 L CNN
+F 0 "J4" H 4630 1492 50  0000 L CNN
 F 1 "Screw_Terminal_Thermo_2" H 4630 1401 50  0000 L CNN
 F 2 "TerminalBlock_Phoenix:TerminalBlock_Phoenix_MPT-0,5-2-2.54_1x02_P2.54mm_Horizontal" H 4550 1500 50  0001 C CNN
@@
 	4400 2100 4400 2250
 $Comp
-L Sensor_Temperature:MAX31855RASA U?
+L Sensor_Temperature:MAX31855RASA U5
 U 1 1 5DAB1C41
 P 4950 2400
-F 0 "U?" H 4950 2981 50  0000 C CNN
+F 0 "U5" H 4950 2981 50  0000 C CNN
 F 1 "MAX31855RASA" H 4950 2890 50  0000 C CNN
 F 2 "Package_SO:SOIC-8_3.9x4.9mm_P1.27mm" H 5950 2050 50  0001 C CIN
@@
 	1    0    0    -1
 $EndComp
+Text Label 4000 1600 0    50   ~ 0
+T2_T+
 Text Label 4000 1500 0    50   ~ 0
-T2_T+
-Text Label 4000 1600 0    50   ~ 0
 T2_T-
 Wire Wire Line
@@
 Text Label 6400 2700 0    50   ~ 0
 T3_T-
+Text Label 6000 1600 0    50   ~ 0
+T3_T+
 Text Label 6000 1500 0    50   ~ 0
-T3_T+
-Text Label 6000 1600 0    50   ~ 0
 T3_T-
 $Comp
-L Connector:Screw_Terminal_01x02 J?
+L Connector:Screw_Terminal_01x02 J5
 U 1 1 5DAE7830
 P 6550 1500
-F 0 "J?" H 6630 1492 50  0000 L CNN
+F 0 "J5" H 6630 1492 50  0000 L CNN
 F 1 "Screw_Terminal_Thermo_3" H 6630 1401 50  0000 L CNN
 F 2 "TerminalBlock_Phoenix:TerminalBlock_Phoenix_MPT-0,5-2-2.54_1x02_P2.54mm_Horizontal" H 6550 1500 50  0001 C CNN
@@
 Text Label 8400 2700 0    50   ~ 0
 T4_T-
+Text Label 8000 1600 0    50   ~ 0
+T4_T+
 Text Label 8000 1500 0    50   ~ 0
-T4_T+
-Text Label 8000 1600 0    50   ~ 0
 T4_T-
 $Comp
-L Connector:Screw_Terminal_01x02 J?
+L Connector:Screw_Terminal_01x02 J6
 U 1 1 5DAEBA70
 P 8550 1500
-F 0 "J?" H 8630 1492 50  0000 L CNN
+F 0 "J6" H 8630 1492 50  0000 L CNN
 F 1 "Screw_Terminal_Thermo_4" H 8630 1401 50  0000 L CNN
 F 2 "TerminalBlock_Phoenix:TerminalBlock_Phoenix_MPT-0,5-2-2.54_1x02_P2.54mm_Horizontal" H 8550 1500 50  0001 C CNN
