File: thermocouples.sch (KiCad schematic (older format))
At the start: 0 parts

Commit message: Update thermocouples.sch
Parts:
- added C? (x4): 100nF, Capacitor_SMD:C_0603_1608Metric, symbol Device:C
- added C? (x4): 10nF, Capacitor_SMD:C_0603_1608Metric, symbol Device:C
- added J?: Screw_Terminal_Thermo_1, TerminalBlock_Phoenix:TerminalBlock_Phoenix_MPT-0,5-2-2.54_1x02_P2.54mm_Horizontal, symbol Connector:Screw_Terminal_01x02
- added J?: Screw_Terminal_Thermo_2, TerminalBlock_Phoenix:TerminalBlock_Phoenix_MPT-0,5-2-2.54_1x02_P2.54mm_Horizontal, symbol Connector:Screw_Terminal_01x02
- added J?: Screw_Terminal_Thermo_3, TerminalBlock_Phoenix:TerminalBlock_Phoenix_MPT-0,5-2-2.54_1x02_P2.54mm_Horizontal, symbol Connector:Screw_Terminal_01x02
- added J?: Screw_Terminal_Thermo_4, TerminalBlock_Phoenix:TerminalBlock_Phoenix_MPT-0,5-2-2.54_1x02_P2.54mm_Horizontal, symbol Connector:Screw_Terminal_01x02
- added U? (x4): MAX31855RASA, Package_SO:SOIC-8_3.9x4.9mm_P1.27mm, symbol Sensor_Temperature:MAX31855RASA
Connections:
- new net +3V3: C?.1, C?.1, C?.1, C?.1, U?.4 (VCC), U?.4 (VCC), U?.4 (VCC), U?.4 (VCC)
- new net GND: C?.2, C?.2, C?.2, C?.2, U?.1 (GND), U?.1 (GND), U?.1 (GND), U?.1 (GND)
- new net MISO: U?.7 (SO), U?.7 (SO), U?.7 (SO), U?.7 (SO)
- new net SCLK: U?.5 (SCK), U?.5 (SCK), U?.5 (SCK), U?.5 (SCK)
- new net T1_T+: C?.1, J?.1 (Pin_1), U?.3 (T+)
- new net T1_T-: C?.2, J?.2 (Pin_2), U?.2 (T-)
- new net T2_T+: C?.1, J?.1 (Pin_1), U?.3 (T+)
- new net T2_T-: C?.2, J?.2 (Pin_2), U?.2 (T-)
- new net T3_T+: C?.1, J?.1 (Pin_1), U?.3 (T+)
- new net T3_T-: C?.2, J?.2 (Pin_2), U?.2 (T-)
- new net T4_T+: C?.1, J?.1 (Pin_1), U?.3 (T+)
- new net T4_T-: C?.2, J?.2 (Pin_2), U?.2 (T-)
- new net ~CS_1: U?.6 (~CS~)
- new net ~CS_2: U?.6 (~CS~)
- new net ~CS_3: U?.6 (~CS~)
- new net ~CS_4: U?.6 (~CS~)

Commit message: amplifier changes
Parts:
- removed C? (x4): 100nF, Capacitor_SMD:C_0603_1608Metric, symbol Device:C
- removed C? (x4): 10nF, Capacitor_SMD:C_0603_1608Metric, symbol Device:C
- removed J?: Screw_Terminal_Thermo_1, TerminalBlock_Phoenix:TerminalBlock_Phoenix_MPT-0,5-2-2.54_1x02_P2.54mm_Horizontal, symbol Connector:Screw_Terminal_01x02
- removed J?: Screw_Terminal_Thermo_2, TerminalBlock_Phoenix:TerminalBlock_Phoenix_MPT-0,5-2-2.54_1x02_P2.54mm_Horizontal, symbol Connector:Screw_Terminal_01x02
- removed J?: Screw_Terminal_Thermo_3, TerminalBlock_Phoenix:TerminalBlock_Phoenix_MPT-0,5-2-2.54_1x02_P2.54mm_Horizontal, symbol Connector:Screw_Terminal_01x02
- removed J?: Screw_Terminal_Thermo_4, TerminalBlock_Phoenix:TerminalBlock_Phoenix_MPT-0,5-2-2.54_1x02_P2.54mm_Horizontal, symbol Connector:Screw_Terminal_01x02
- removed U? (x4): MAX31855RASA, Package_SO:SOIC-8_3.9x4.9mm_P1.27mm, symbol Sensor_Temperature:MAX31855RASA
