File: thermocouples.sch (KiCad schematic (older format))
At the start: 16 parts, among them J6 Screw_Terminal_Thermo_1, J7 Screw_Terminal_Thermo_2, J8 Screw_Terminal_Thermo_3, J9 Screw_Terminal_Thermo_4, U6 MAX31855RASA, U7 MAX31855RASA, U8 MAX31855RASA, U9 MAX31855RASA

Commit message: Fixed conflicts, assigned all footprints.
Parts:
- renumbered C9 to C15, C10 to C16, C11 to C17, C12 to C18, C13 to C19, C14 to C20, C15 to C21, C16 to C22, J6 to J5, J7 to J6, J8 to J7, J9 to J8
Changed lines of the file:
@@
 $Descr A4 11693 8268
 encoding utf-8
-Sheet 5 6
+Sheet 3 5
 Title ""
 Date ""
@@
 $EndComp
 $Comp
-L Device:C C9
+L Device:C C15
 U 1 1 5DA633EE
 P 2000 2400
-F 0 "C9" H 2115 2446 50  0000 L CNN
+F 0 "C15" H 2115 2446 50  0000 L CNN
 F 1 "100nF" H 2115 2355 50  0000 L CNN
 F 2 "Capacitor_SMD:C_0603_1608Metric" H 2038 2250 50  0001 C CNN
@@
 	2000 2000 2000 2250
 $Comp
-L power:+3V3 #PWR0145
+L power:+3V3 #PWR043
 U 1 1 5DA64666
 P 2000 1900
-F 0 "#PWR0145" H 2000 1750 50  0001 C CNN
+F 0 "#PWR043" H 2000 1750 50  0001 C CNN
 F 1 "+3V3" H 2015 2073 50  0000 C CNN
 F 2 "" H 2000 1900 50  0001 C CNN
@@
 Connection ~ 2000 2000
 $Comp
-L power:GND #PWR0146
+L power:GND #PWR044
 U 1 1 5DA65041
 P 2000 2900
-F 0 "#PWR0146" H 2000 2650 50  0001 C CNN
+F 0 "#PWR044" H 2000 2650 50  0001 C CNN
 F 1 "GND" H 2005 2727 50  0000 C CNN
 F 2 "" H 2000 2900 50  0001 C CNN
@@
 Connection ~ 2000 2800
 $Comp
-L Device:C C10
+L Device:C C16
 U 1 1 5DA6662C
 P 2400 2400
-F 0 "C10" H 2515 2446 50  0000 L CNN
+F 0 "C16" H 2515 2446 50  0000 L CNN
 F 1 "10nF" H 2515 2355 50  0000 L CNN
 F 2 "Capacitor_SMD:C_0603_1608Metric" H 2438 2250 50  0001 C CNN
@@
 $EndComp
 $Comp
-L Device:C C13
+L Device:C C19
 U 1 1 5DAB0490
 P 6000 2400
-F 0 "C13" H 6115 2446 50  0000 L CNN
+F 0 "C19" H 6115 2446 50  0000 L CNN
 F 1 "100nF" H 6115 2355 50  0000 L CNN
 F 2 "Capacitor_SMD:C_0603_1608Metric" H 6038 2250 50  0001 C CNN
@@
 	6000 2000 6000 2250
 $Comp
-L power:+3V3 #PWR0147
+L power:+3V3 #PWR047
 U 1 1 5DAB049A
 P 6000 1900
-F 0 "#PWR0147" H 6000 1750 50  0001 C CNN
+F 0 "#PWR047" H 6000 1750 50  0001 C CNN
 F 1 "+3V3" H 6015 2073 50  0000 C CNN
 F 2 "" H 6000 1900 50  0001 C CNN
@@
 Connection ~ 6000 2000
 $Comp
-L power:GND #PWR0148
+L power:GND #PWR048
 U 1 1 5DAB04A2
 P 6000 2900
-F 0 "#PWR0148" H 6000 2650 50  0001 C CNN
+F 0 "#PWR048" H 6000 2650 50  0001 C CNN
 F 1 "GND" H 6005 2727 50  0000 C CNN
 F 2 "" H 6000 2900 50  0001 C CNN
@@
 Connection ~ 6000 2800
 $Comp
-L Device:C C14
+L Device:C C20
 U 1 1 5DAB04AA
 P 6400 2400
-F 0 "C14" H 6515 2446 50  0000 L CNN
+F 0 "C20" H 6515 2446 50  0000 L CNN
 F 1 "10nF" H 6515 2355 50  0000 L CNN
 F 2 "Capacitor_SMD:C_0603_1608Metric" H 6438 2250 50  0001 C CNN
@@
 	6550 2550 6400 2550
 $Comp
-L Device:C C11
+L Device:C C17
 U 1 1 5DAB1C47
 P 4000 2400
-F 0 "C11" H 4115 2446 50  0000 L CNN
+F 0 "C17" H 4115 2446 50  0000 L CNN
 F 1 "100nF" H 4115 2355 50  0000 L CNN
 F 2 "Capacitor_SMD:C_0603_1608Metric" H 4038 2250 50  0001 C CNN
@@
 	4000 2000 4000 2250
 $Comp
-L power:+3V3 #PWR0149
+L power:+3V3 #PWR045
 U 1 1 5DAB1C51
 P 4000 1900
-F 0 "#PWR0149" H 4000 1750 50  0001 C CNN
+F 0 "#PWR045" H 4000 1750 50  0001 C CNN
 F 1 "+3V3" H 4015 2073 50  0000 C CNN
 F 2 "" H 4000 1900 50  0001 C CNN
@@
 Connection ~ 4000 2000
 $Comp
-L power:GND #PWR0150
+L power:GND #PWR046
 U 1 1 5DAB1C59
 P 4000 2900
-F 0 "#PWR0150" H 4000 2650 50  0001 C CNN
+F 0 "#PWR046" H 4000 2650 50  0001 C CNN
 F 1 "GND" H 4005 2727 50  0000 C CNN
 F 2 "" H 4000 2900 50  0001 C CNN
@@
 Connection ~ 4000 2800
 $Comp
-L Device:C C12
+L Device:C C18
 U 1 1 5DAB1C61
 P 4400 2400
-F 0 "C12" H 4515 2446 50  0000 L CNN
+F 0 "C18" H 4515 2446 50  0000 L CNN
 F 1 "10nF" H 4515 2355 50  0000 L CNN
 F 2 "Capacitor_SMD:C_0603_1608Metric" H 4438 2250 50  0001 C CNN
@@
 $EndComp
 $Comp
-L Device:C C15
+L Device:C C21
 U 1 1 5DAC219C
 P 8000 2400
-F 0 "C15" H 8115 2446 50  0000 L CNN
+F 0 "C21" H 8115 2446 50  0000 L CNN
 F 1 "100nF" H 8115 2355 50  0000 L CNN
 F 2 "Capacitor_SMD:C_0603_1608Metric" H 8038 2250 50  0001 C CNN
@@
 	8000 2000 8000 2250
 $Comp
-L power:+3V3 #PWR0151
+L power:+3V3 #PWR049
 U 1 1 5DAC21A6
 P 8000 1900
-F 0 "#PWR0151" H 8000 1750 50  0001 C CNN
+F 0 "#PWR049" H 8000 1750 50  0001 C CNN
 F 1 "+3V3" H 8015 2073 50  0000 C CNN
 F 2 "" H 8000 1900 50  0001 C CNN
@@
 Connection ~ 8000 2000
 $Comp
-L power:GND #PWR0152
+L power:GND #PWR050
 U 1 1 5DAC21AE
 P 8000 2900
-F 0 "#PWR0152" H 8000 2650 50  0001 C CNN
+F 0 "#PWR050" H 8000 2650 50  0001 C CNN
 F 1 "GND" H 8005 2727 50  0000 C CNN
 F 2 "" H 8000 2900 50  0001 C CNN
@@
 Connection ~ 8000 2800
 $Comp
-L Device:C C16
+L Device:C C22
 U 1 1 5DAC21B6
 P 8400 2400
-F 0 "C16" H 8515 2446 50  0000 L CNN
+F 0 "C22" H 8515 2446 50  0000 L CNN
 F 1 "10nF" H 8515 2355 50  0000 L CNN
 F 2 "Capacitor_SMD:C_0603_1608Metric" H 8438 2250 50  0001 C CNN
@@
 Text HLabel 9350 2200 2    50   Input ~ 0
 SCLK
-Text HLabel 9350 2300 2    50   Input ~ 0
-MISO
 Text HLabel 9350 2500 2    50   Input ~ 0
 ~CS_4
@@
 Text Label 2000 1500 0    50   ~ 0
 T1_T-
-$Comp
-L Connector:Screw_Terminal_01x02 J6
-U 1 1 5DAD8258
-P 2550 1500
-F 0 "J6" H 2630 1492 50  0000 L CNN
-F 1 "Screw_Terminal_Thermo_1" H 2630 1401 50  0000 L CNN
-F 2 "TerminalBlock_Phoenix:TerminalBlock_Phoenix_MPT-0,5-2-2.54_1x02_P2.54mm_Horizontal" H 2550 1500 50  0001 C CNN
-F 3 "~" H 2550 1500 50  0001 C CNN
-	1    2550 1500
-	1    0    0    -1
-$EndComp
 Text Label 2400 2100 0    50   ~ 0
 T1_T+
@@
 Text Label 4400 2700 0    50   ~ 0
 T2_T-
-$Comp
-L Connector:Screw_Terminal_01x02 J7
-U 1 1 5DAE1281
-P 4550 1500
-F 0 "J7" H 4630 1492 50  0000 L CNN
-F 1 "Screw_Terminal_Thermo_2" H 4630 1401 50  0000 L CNN
-F 2 "TerminalBlock_Phoenix:TerminalBlock_Phoenix_MPT-0,5-2-2.54_1x02_P2.54mm_Horizontal" H 4550 1500 50  0001 C CNN
-F 3 "~" H 4550 1500 50  0001 C CNN
-	1    4550 1500
-	1    0    0    -1
-$EndComp
 Connection ~ 4400 2250
 Wire Wire Line
@@
 Text Label 6000 1500 0    50   ~ 0
 T3_T-
-$Comp
-L Connector:Screw_Terminal_01x02 J8
-U 1 1 5DAE7830
-P 6550 1500
-F 0 "J8" H 6630 1492 50  0000 L CNN
-F 1 "Screw_Terminal_Thermo_3" H 6630 1401 50  0000 L CNN
-F 2 "TerminalBlock_Phoenix:TerminalBlock_Phoenix_MPT-0,5-2-2.54_1x02_P2.54mm_Horizontal" H 6550 1500 50  0001 C CNN
-F 3 "~" H 6550 1500 50  0001 C CNN
-	1    6550 1500
-	1    0    0    -1
-$EndComp
 Wire Wire Line
 	6000 1500 6350 1500
@@
 Text Label 8000 1500 0    50   ~ 0
 T4_T-
-$Comp
-L Connector:Screw_Terminal_01x02 J9
+Wire Wire Line
+	8000 1500 8350 1500
+Wire Wire Line
+	8000 1600 8350 1600
+Wire Wire Line
+	2000 1500 2350 1500
+Wire Wire Line
+	2000 1600 2350 1600
+Text HLabel 7350 2200 2    50   Input ~ 0
+SCLK
+Text HLabel 5350 2200 2    50   Input ~ 0
+SCLK
+Text HLabel 3350 2200 2    50   Input ~ 0
+SCLK
+Text HLabel 3350 2300 2    50   Output ~ 0
+MISO
+Text HLabel 5350 2300 2    50   Output ~ 0
+MISO
+Text HLabel 7350 2300 2    50   Output ~ 0
+MISO
+Text HLabel 9350 2300 2    50   Output ~ 0
+MISO
+$Comp
+L Connector:Screw_Terminal_01x02 J8
 U 1 1 5DAEBA70
 P 8550 1500
-F 0 "J9" H 8630 1492 50  0000 L CNN
+F 0 "J8" H 8630 1492 50  0000 L CNN
 F 1 "Screw_Terminal_Thermo_4" H 8630 1401 50  0000 L CNN
 F 2 "TerminalBlock_Phoenix:TerminalBlock_Phoenix_MPT-0,5-2-2.54_1x02_P2.54mm_Horizontal" H 8550 1500 50  0001 C CNN
@@
 	1    0    0    -1
 $EndComp
-Wire Wire Line
-	8000 1500 8350 1500
-Wire Wire Line
-	8000 1600 8350 1600
-Wire Wire Line
-	2000 1500 2350 1500
-Wire Wire Line
-	2000 1600 2350 1600
-Text HLabel 7350 2200 2    50   Input ~ 0
-SCLK
-Text HLabel 7350 2300 2    50   Input ~ 0
-MISO
-Text HLabel 5350 2200 2    50   Input ~ 0
-SCLK
-Text HLabel 5350 2300 2    50   Input ~ 0
-MISO
-Text HLabel 3350 2200 2    50   Input ~ 0
-SCLK
-Text HLabel 3350 2300 2    50   Input ~ 0
-MISO
+$Comp
+L Connector:Screw_Terminal_01x02 J7
+U 1 1 5DAE7830
+P 6550 1500
+F 0 "J7" H 6630 1492 50  0000 L CNN
+F 1 "Screw_Terminal_Thermo_3" H 6630 1401 50  0000 L CNN
+F 2 "TerminalBlock_Phoenix:TerminalBlock_Phoenix_MPT-0,5-2-2.54_1x02_P2.54mm_Horizontal" H 6550 1500 50  0001 C CNN
+F 3 "~" H 6550 1500 50  0001 C CNN
+	1    6550 1500
+	1    0    0    -1
+$EndComp
+$Comp
+L Connector:Screw_Terminal_01x02 J6
+U 1 1 5DAE1281
+P 4550 1500
+F 0 "J6" H 4630 1492 50  0000 L CNN
+F 1 "Screw_Terminal_Thermo_2" H 4630 1401 50  0000 L CNN
+F 2 "TerminalBlock_Phoenix:TerminalBlock_Phoenix_MPT-0,5-2-2.54_1x02_P2.54mm_Horizontal" H 4550 1500 50  0001 C CNN
+F 3 "~" H 4550 1500 50  0001 C CNN
+	1    4550 1500
+	1    0    0    -1
+$EndComp
+$Comp
+L Connector:Screw_Terminal_01x02 J5
+U 1 1 5DAD8258
+P 2550 1500
+F 0 "J5" H 2630 1492 50  0000 L CNN
+F 1 "Screw_Terminal_Thermo_1" H 2630 1401 50  0000 L CNN
+F 2 "TerminalBlock_Phoenix:TerminalBlock_Phoenix_MPT-0,5-2-2.54_1x02_P2.54mm_Horizontal" H 2550 1500 50  0001 C CNN
+F 3 "~" H 2550 1500 50  0001 C CNN
+	1    2550 1500
+	1    0    0    -1
+$EndComp
 $EndSCHEMATC

Commit message: Cleaned up layout, added barrel jack for power input
Parts:
- J5, J6, J7, J8: footprint TerminalBlock_Phoenix:TerminalBlock_Phoenix_MPT-0,5-2-2.54_1x02_P2.54mm_Horizontal -> TerminalBlock_Phoenix:TerminalBlock_Phoenix_MPT-2.54mm_2pol
Connections:
- net ~CS_2: now also U7.6 (~CS~); no longer U8.6 (~CS~)
- net ~CS_3: now also U8.6 (~CS~); no longer U7.6 (~CS~)
Changed lines of the file:
@@
 ~CS_1
 Text HLabel 7350 2500 2    50   Input ~ 0
+~CS_3
+Text HLabel 5350 2500 2    50   Input ~ 0
 ~CS_2
-Text HLabel 5350 2500 2    50   Input ~ 0
-~CS_3
 Text HLabel 9350 2200 2    50   Input ~ 0
 SCLK
@@
 F 0 "J8" H 8630 1492 50  0000 L CNN
 F 1 "Screw_Terminal_Thermo_4" H 8630 1401 50  0000 L CNN
-F 2 "TerminalBlock_Phoenix:TerminalBlock_Phoenix_MPT-0,5-2-2.54_1x02_P2.54mm_Horizontal" H 8550 1500 50  0001 C CNN
+F 2 "TerminalBlock_Phoenix:TerminalBlock_Phoenix_MPT-2.54mm_2pol" H 8550 1500 50  0001 C CNN
 F 3 "~" H 8550 1500 50  0001 C CNN
 	1    8550 1500
@@
 F 0 "J7" H 6630 1492 50  0000 L CNN
 F 1 "Screw_Terminal_Thermo_3" H 6630 1401 50  0000 L CNN
-F 2 "TerminalBlock_Phoenix:TerminalBlock_Phoenix_MPT-0,5-2-2.54_1x02_P2.54mm_Horizontal" H 6550 1500 50  0001 C CNN
+F 2 "TerminalBlock_Phoenix:TerminalBlock_Phoenix_MPT-2.54mm_2pol" H 6550 1500 50  0001 C CNN
 F 3 "~" H 6550 1500 50  0001 C CNN
 	1    6550 1500
@@
 F 0 "J6" H 4630 1492 50  0000 L CNN
 F 1 "Screw_Terminal_Thermo_2" H 4630 1401 50  0000 L CNN
-F 2 "TerminalBlock_Phoenix:TerminalBlock_Phoenix_MPT-0,5-2-2.54_1x02_P2.54mm_Horizontal" H 4550 1500 50  0001 C CNN
+F 2 "TerminalBlock_Phoenix:TerminalBlock_Phoenix_MPT-2.54mm_2pol" H 4550 1500 50  0001 C CNN
 F 3 "~" H 4550 1500 50  0001 C CNN
 	1    4550 1500
@@
 F 0 "J5" H 2630 1492 50  0000 L CNN
 F 1 "Screw_Terminal_Thermo_1" H 2630 1401 50  0000 L CNN
-F 2 "TerminalBlock_Phoenix:TerminalBlock_Phoenix_MPT-0,5-2-2.54_1x02_P2.54mm_Horizontal" H 2550 1500 50  0001 C CNN
+F 2 "TerminalBlock_Phoenix:TerminalBlock_Phoenix_MPT-2.54mm_2pol" H 2550 1500 50  0001 C CNN
 F 3 "~" H 2550 1500 50  0001 C CNN
 	1    2550 1500
