File: daq-hardware.sch (KiCad schematic (older format))
At the start: 9 parts, among them J1 USB_B, J2 Micro_SD_Card_Det_Hirose_DM3AT, Q1 MMDT2222A, U1 CP2102N-A01-GQFN24, U2 ESP32-WROOM-32D

Commit message: Fixed Main schem and removed baro
Parts:
- added C?: 0.1uF, symbol Device:C_Small
- added C? (x2): 1nF, symbol Device:C_Small
- added R? (x2): 10k, symbol Device:R_Small
- added R? (x2): 470, symbol Device:R_Small
- added SW? (x2): SW1, symbol Switch:SW_Push
Connections:
- net +3V3: now also R?.1, R?.1
- net GND: now also C?.2, C?.2, C?.2, SW?.1, SW?.1
- net GPIO0: now also R?.1, R?.2
- net RESET: now also C?.1, R?.1, R?.2
- net SD_CS: now reaches U2.29 (IO5)
- net SD_CS: now also J2.2 (DAT3/CD)
- net SCLK: now reaches U2.30 (IO18)
- net SCLK: now also J2.5 (CLK)
- net MISO: now reaches U2.31 (IO19)
- net MISO: now also J2.7 (DAT0)
- net MOSI: now reaches U2.37 (IO23)
- net MOSI: now also J2.3 (CMD)
- net BARO_CS: now reaches U2.6 (IO34)
- new net: C?.1, R?.2, SW?.2 (x2)
- no-connect marks 7 -> 11
Other:
- moved on the sheet: J1, Q1A, Q1B, R1, R2, R3, R4, U1
