File: power.sch (KiCad schematic (older format))
At the start: 28 parts

Commit message: added inductors footprint
Parts:
- L? (x3): footprint (none) -> Inductor_SMD:L_Taiyo-Yuden_NR-30xx
Changed lines of the file:
@@
 F 0 "L?" H 4250 1415 50  0000 C CNN
 F 1 "2u2" H 4250 1324 50  0000 C CNN
-F 2 "" H 4250 1323 50  0001 C CNN
+F 2 "Inductor_SMD:L_Taiyo-Yuden_NR-30xx" H 4250 1323 50  0001 C CNN
 F 3 "~" H 4250 1200 50  0001 C CNN
 	1    4250 1200
@@
 F 0 "L?" H 4250 2965 50  0000 C CNN
 F 1 "2u2" H 4250 2874 50  0000 C CNN
-F 2 "" H 4250 2873 50  0001 C CNN
+F 2 "Inductor_SMD:L_Taiyo-Yuden_NR-30xx" H 4250 2873 50  0001 C CNN
 F 3 "~" H 4250 2750 50  0001 C CNN
 	1    4250 2750
@@
 F 0 "L?" H 3250 4465 50  0000 C CNN
 F 1 "10u" H 3250 4374 50  0000 C CNN
-F 2 "" H 3250 4250 50  0001 C CNN
+F 2 "Inductor_SMD:L_Taiyo-Yuden_NR-30xx" H 3250 4250 50  0001 C CNN
 F 3 "~" H 3250 4250 50  0001 C CNN
 	1    3250 4250
