File: analogue.sch (KiCad schematic (older format))
At the start: 15 parts, among them J11 Screw_Terminal_01x01, J12 Screw_Terminal_01x01, J13 Screw_Terminal_01x01, J14 Screw_Terminal_01x01, U11 ADS131M04

Commit message: layout changes
Parts:
- U11: symbol iclr:ADS131M04 -> daq-hardware-rescue:ADS131M04-iclr
Changed lines of the file:
@@
 	6200 3600 6650 3600
 $Comp
-L iclr:ADS131M04 U11
+L daq-hardware-rescue:ADS131M04-iclr U11
 U 1 1 5DB46B47
 P 5700 3750
+AR Path="/5DB46B47" Ref="U11"  Part="1"
+AR Path="/5DA926B9/5DB46B47" Ref="U11"  Part="1"
 F 0 "U11" H 5700 4425 50  0000 C CNN
 F 1 "ADS131M04" H 5700 4334 50  0000 C CNN

Commit message: Release candidate
Parts:
- C27: footprint Capacitor_SMD:C_0201_0603Metric -> Capacitor_SMD:C_0603_1608Metric_Pad1.05x0.95mm_HandSolder
Changed lines of the file:
@@
 $Descr A4 11693 8268
 encoding utf-8
-Sheet 5 6
+Sheet 5 7
 Title ""
 Date ""
@@
 F 0 "C27" V 6198 3500 50  0000 C CNN
 F 1 "220nF" V 6289 3500 50  0000 C CNN
-F 2 "Capacitor_SMD:C_0201_0603Metric" H 6488 3350 50  0001 C CNN
+F 2 "Capacitor_SMD:C_0603_1608Metric_Pad1.05x0.95mm_HandSolder" H 6488 3350 50  0001 C CNN
 F 3 "~" H 6450 3500 50  0001 C CNN
 	1    6450 3500

Commit message: Edward appeasement
Parts:
- added C?: 100n, Capacitor_SMD:C_0603_1608Metric, symbol Device:C
Connections:
- net +3V3: now also C?.2
- net GND: now also C?.1
Changed lines of the file:
@@
 Wire Wire Line
 	7250 4200 7250 3900
+$Comp
+L Device:C C?
+U 1 1 5E1BAB7F
+P 7800 3750
+F 0 "C?" H 7915 3796 50  0000 L CNN
+F 1 "100n" H 7915 3705 50  0000 L CNN
+F 2 "Capacitor_SMD:C_0603_1608Metric" H 7838 3600 50  0001 C CNN
+F 3 "~" H 7800 3750 50  0001 C CNN
+	1    7800 3750
+	1    0    0    1
+$EndComp
+$Comp
+L power:+3V3 #PWR?
+U 1 1 5E1BB1FA
+P 7800 3550
+F 0 "#PWR?" H 7800 3400 50  0001 C CNN
+F 1 "+3V3" H 7815 3723 50  0000 C CNN
+F 2 "" H 7800 3550 50  0001 C CNN
+F 3 "" H 7800 3550 50  0001 C CNN
+	1    7800 3550
+	1    0    0    -1
+$EndComp
+$Comp
+L power:GND #PWR?
+U 1 1 5E1BB739
+P 7800 3950
+F 0 "#PWR?" H 7800 3700 50  0001 C CNN
+F 1 "GND" H 7805 3777 50  0000 C CNN
+F 2 "" H 7800 3950 50  0001 C CNN
+F 3 "" H 7800 3950 50  0001 C CNN
+	1    7800 3950
+	1    0    0    -1
+$EndComp
+Wire Wire Line
+	7800 3950 7800 3900
+Wire Wire Line
+	7800 3600 7800 3550
 $EndSCHEMATC
