File: daq-hardware.kicad_pcb (KiCad board)
At the start: 4 copper layers, 100 x 60 mm, 116 parts, among them J1 USB_B, J10 Screw_Terminal_01x02, J11 Screw_Terminal_01x01, J12 Screw_Terminal_01x01, J13 Screw_Terminal_01x01, J14 Screw_Terminal_01x01, J15 Barrel_Jack_Switch, J16 Conn_01x03, J17 Conn_01x03, J18 Conn_01x03, J2 Micro_SD_Card_Det_Hirose_DM3AT, J3 Conn_01x02, J4 Screw_Terminal_01x02, J5 Screw_Terminal_Thermo_1, J6 Screw_Terminal_Thermo_2, J7 Screw_Terminal_Thermo_3, J8 Screw_Terminal_Thermo_4, J9 Screw_Terminal_01x02, Q1 MMDT2222A, Q2 PMV20ENR, Q3 PMV20ENR, SW1 SW1, SW2 SW1, U1 CP2102N-A01-GQFN24, U10 LTV-817S, U11 ADS131M04, U13 TPS2412PW, U2 ESP32-WROOM-32D, U3 TPS61093, U4 TPS62160DGK, U5 TPS62160DGK, U6 MAX31855RASA, U7 MAX31855RASA, U8 MAX31855RASA, U9 MAX31855RASA

Commit message: Release candidate
Parts:
- added C29: 10u, Capacitor_SMD:CP_Elec_4x5.4, F.Cu at (146.9, 99.0)
- added C30: 10u, Capacitor_SMD:CP_Elec_4x5.4, F.Cu at (142.0, 99.0)
- added C31: 10u, Capacitor_SMD:CP_Elec_4x5.4, F.Cu at (183.7, 127.7)
- added J19: Conn_01x03, Connector_PinHeader_2.54mm:PinHeader_1x03_P2.54mm_Vertical, F.Cu at (192.7, 128.2)
- added J20: Conn_01x03, Connector_PinHeader_2.54mm:PinHeader_1x03_P2.54mm_Vertical, F.Cu at (192.7, 125.7)
- added J21: Conn_01x03, Connector_PinHeader_2.54mm:PinHeader_1x03_P2.54mm_Vertical, F.Cu at (192.7, 123.1)
- added J22: Conn_01x03, Connector_PinHeader_2.54mm:PinHeader_1x03_P2.54mm_Vertical, F.Cu at (192.7, 120.6)
- added J23: Conn_01x03, Connector_PinHeader_2.54mm:PinHeader_1x03_P2.54mm_Vertical, F.Cu at (192.7, 118.0)
- added J24: Conn_01x03, Connector_PinHeader_2.54mm:PinHeader_1x03_P2.54mm_Vertical, F.Cu at (192.7, 115.5)
- added J25: Conn_01x03, Connector_PinHeader_2.54mm:PinHeader_1x03_P2.54mm_Vertical, F.Cu at (192.7, 113.0)
- added J26: Conn_01x03, Connector_PinHeader_2.54mm:PinHeader_1x03_P2.54mm_Vertical, F.Cu at (192.7, 110.4)
- added J27: Conn_01x03, Connector_PinHeader_2.54mm:PinHeader_1x03_P2.54mm_Vertical, F.Cu at (192.7, 107.9)
- added J28: Conn_01x03, Connector_PinHeader_2.54mm:PinHeader_1x03_P2.54mm_Vertical, F.Cu at (192.7, 105.3)
- added J29: Conn_01x03, Connector_PinHeader_2.54mm:PinHeader_1x03_P2.54mm_Vertical, F.Cu at (192.7, 102.8)
- added J30: Conn_01x03, Connector_PinHeader_2.54mm:PinHeader_1x03_P2.54mm_Vertical, F.Cu at (192.7, 100.2)
- added J31: Conn_01x03, Connector_PinHeader_2.54mm:PinHeader_1x03_P2.54mm_Vertical, F.Cu at (192.7, 97.7)
- added J32: Conn_01x03, Connector_PinHeader_2.54mm:PinHeader_1x03_P2.54mm_Vertical, F.Cu at (192.7, 95.2)
- added J33: Conn_01x03, Connector_PinHeader_2.54mm:PinHeader_1x03_P2.54mm_Vertical, F.Cu at (192.7, 92.6)
- added J34: Conn_01x03, Connector_PinHeader_2.54mm:PinHeader_1x03_P2.54mm_Vertical, F.Cu at (192.7, 130.7)
- added J35: Conn_01x04, Connector_PinHeader_2.54mm:PinHeader_1x04_P2.54mm_Vertical, F.Cu at (179.2, 119.4)
- added J36: Screw_Terminal_01x02, TerminalBlock_Phoenix:TerminalBlock_Phoenix_MPT-2.54mm_2pol, F.Cu at (181.2, 136.8)
- added J37: Screw_Terminal_01x02, TerminalBlock_Phoenix:TerminalBlock_Phoenix_MPT-2.54mm_2pol, F.Cu at (188.2, 136.8)
- added JP3: Jumper, Connector_PinHeader_2.54mm:PinHeader_1x02_P2.54mm_Vertical, F.Cu at (162.6, 131.4)
- added SW3: SW_DPDT_x2, Button_Switch_THT:SW_CuK_JS202011AQN_DPDT_Angled, F.Cu at (172.6, 83.8)
- added U12: PCA9685PW, Package_SO:TSSOP-28_4.4x9.7mm_P0.65mm, F.Cu at (183.2, 110.2)
- added U2 (x2): ESP32-WROOM-32D, RF_Module:ESP32-WROOM-32U, F.Cu at (110.0, 110.5)
- C11, C13: value 10u -> 100n; footprint Capacitor_SMD:CP_Elec_4x5.4 -> Capacitor_SMD:C_0603_1608Metric
- C27: footprint Capacitor_SMD:C_0201_0603Metric -> Capacitor_SMD:C_0603_1608Metric_Pad1.05x0.95mm_HandSolder
- D1: footprint Diode_SMD:D_0603_1608Metric_Castellated -> LED_SMD:LED_0603_1608Metric_Castellated
- D3, D7: footprint LED_SMD:LED_0805_2012Metric -> LED_SMD:LED_0603_1608Metric_Castellated
- L2, L3: value 2u2 -> 1u5
- R1, R6: value 10k -> 4k7
- R16: value 230k -> 191k
- R19, R20: value 100k -> 10k
- R21: value 62k5 -> 100k
- R22: value 52k5 -> 100k
- R23: value 20k -> 470k
- R24: value 10k -> 150k
- U2: footprint RF_Module:ESP32-WROOM-32 -> RF_Module:ESP32-WROOM-32U
- U4: value TPS62160DGK -> TPS63070; footprint Housings_SSOP:VSSOP-8_3.0x3.0mm_Pitch0.65mm -> iclr-fp:Texas_PowerVFQFN_15
- U5: value TPS62160DGK -> TPS630701; footprint Housings_SSOP:VSSOP-8_3.0x3.0mm_Pitch0.65mm -> iclr-fp:Texas_PowerVFQFN_15
- moved R29 64.7 mm to (188.5, 90.5)
- moved D7 64.2 mm to (188.5, 89.0), turned to 180 degrees
- moved C1 59.2 mm to (183.4, 116.2)
- moved R1 53.4 mm to (178.0, 115.1), turned to 90 degrees
- moved R6 52.8 mm to (178.0, 112.0), turned to 270 degrees
- moved R17 38.1 mm to (178.0, 126.2)
- moved J10 36.9 mm to (188.0, 83.4), turned to 180 degrees
- moved R18 36.2 mm to (175.6, 127.0), turned to 180 degrees
- moved SW2 35.6 mm to (119.9, 93.5), turned to 270 degrees
- moved R16 34.5 mm to (178.0, 123.0), turned to 270 degrees
- moved C9 34.4 mm to (179.6, 123.0), turned to 90 degrees
- moved C8 34.0 mm to (175.6, 125.2), turned to 180 degrees
- moved C3 33.1 mm to (117.2, 92.2), turned to 270 degrees
- moved J9 32.1 mm to (180.7, 83.4), turned to 180 degrees
- moved R8 29.9 mm to (118.8, 97.3), turned to 0 degrees
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Connections:
- net +12V renamed +10V
- net /SD_CMD renamed /SD_MOSI
- net /SD_D0 renamed /SD_MISO
- net /SD_D3 renamed /SD_CS
- C1 pad 1: /RESET -> GND
- C1 pad 2: GND -> +3V3
- C11 pad 1: +3V3 -> Net-(C11-Pad1)
- C13 pad 1: +3V3 -> Net-(C13-Pad1)
- C5 pad 1: +3V3 -> VDD
- C6 pad 1: +3V3 -> +5V
- JP1 pad 2: Net-(D3-Pad2) -> Net-(JP1-Pad2)
- L1 pad 1: +3V3 -> +5V
- L2 pad 2: +3V3 -> Net-(L2-Pad2)
- L3 pad 2: +5V -> Net-(L3-Pad2)
- R1 pad 2: /RESET -> /SDA
- R19 pad 1: +3V3 -> Net-(R19-Pad1)
- R19 pad 2: /power/PG -> VDD
- R20 pad 1: +5V -> Net-(R20-Pad1)
- R20 pad 2: /power/PG -> VDD
- R21 pad 1: Net-(R21-Pad1) -> +3V3
- R21 pad 2: +3V3 -> Net-(R21-Pad2)
- R22 pad 1: Net-(R22-Pad1) -> +5V
- R22 pad 2: +5V -> Net-(R22-Pad2)
- R23 pad 1: GND -> +3V3
- R23 pad 2: Net-(R21-Pad1) -> /power/FB_3V3
- R24 pad 1: GND -> /power/FB_3V3
- R24 pad 2: Net-(R22-Pad1) -> GND
- R30 pad 2: /ptaps/PTAP1 -> /PTAP1
- R31 pad 1: /ptaps/PTAP1 -> /PTAP1
- R32 pad 2: /ptaps/PTAP2 -> /PTAP2
- R33 pad 1: /ptaps/PTAP2 -> /PTAP2
- R34 pad 2: /ptaps/PTAP3 -> /PTAP3
- R35 pad 1: /ptaps/PTAP3 -> /PTAP3
- R6 pad 2: (no net) -> /SCL
- U11 pad 12: (no net) -> /~ADC_CS
- U2 pad 14: /SD_D2 -> /PYRO
- U2 pad 17: (no net) -> Net-(U2-Pad17)
- U2 pad 18: (no net) -> Net-(U2-Pad18)
- U2 pad 19: (no net) -> Net-(U2-Pad19)
- U2 pad 20: (no net) -> Net-(U2-Pad20)
- U2 pad 21: (no net) -> Net-(U2-Pad21)
- U2 pad 22: (no net) -> Net-(U2-Pad22)
- U2 pad 26: /SD_D1 -> /CONT
- U2 pad 27: (no net) -> /~ADC_CS
- U2 pad 32: (no net) -> Net-(U2-Pad32)
- U2 pad 33: /PYRO -> /SDA
- U2 pad 36: /CONT -> /SCL
- U2 pad 4: (no net) -> Net-(U2-Pad4)
- U2 pad 5: (no net) -> Net-(U2-Pad5)
- U2 pad 6: (no net) -> /PTAP3
- U2 pad 7: (no net) -> /PTAP2
- U2 pad 9: (no net) -> /PTAP1
- U3 pad 11: (no net) -> GND
- U3 pad 2: +3V3 -> +5V
- U3 pad 5: +3V3 -> +5V
- U4 pad 1: GND -> Net-(R19-Pad1)
- U4 pad 2: VDD -> Net-(R21-Pad2)
- U4 pad 3: VDD -> Net-(C11-Pad1)
- U4 pad 5: Net-(R21-Pad1) -> /power/FB_3V3
- U4 pad 6: +3V3 -> GND
- U5 pad 1: GND -> Net-(R20-Pad1)
- U5 pad 2: +3V3 -> Net-(R22-Pad2)
- U5 pad 3: +3V3 -> Net-(C13-Pad1)
- U5 pad 5: Net-(R22-Pad1) -> +5V
- U5 pad 6: +5V -> GND
Routing:
- net +5V: track 2.72 -> 151.1 mm, vias 4 -> 19
- net /SCL: track 0.00 -> 91.8 mm, vias 0 -> 2
- net /SDA: track 0.00 -> 84.5 mm, vias 0 -> 2
- net /~ADC_CS: track 0.00 -> 55.5 mm
- net /PTAP3: track 0.00 -> 50.6 mm, vias 0 -> 2
- net /PTAP2: track 0.00 -> 42.9 mm, vias 0 -> 2
- net Net-(D4-Pad2): track 61.8 -> 24.1 mm, vias 3 -> 1
- net /PTAP1: track 0.00 -> 36.3 mm, vias 0 -> 2
- net /SD_D1: track 35.7 -> 2.65 mm, vias 2 -> 1
- net /BOOT: track 40.9 -> 9.75 mm, vias 2 -> 0
- net /power/PG: track 28.9 -> 0.00 mm
- net /servos/SERVO15: track 0.00 -> 28.7 mm
- net /RESET: track 57.2 -> 30.0 mm, vias 3 -> 2
- net /servos/SERVO14: track 0.00 -> 26.5 mm
- net /servos/SERVO13: track 0.00 -> 24.2 mm
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- added copper zone on F.Cu, net Net-(L2-Pad2)
- added copper zone on F.Cu, net Net-(L3-Pad2)
- removed copper zone on F.Cu, net /power/VO
- removed copper zone on F.Cu, net Net-(C7-Pad1)
- removed copper zone on F.Cu, net Net-(C7-Pad2)
Other:
- board text added: "-: White/Red +: Green/Yellow"
- board text added: "-Vpyro+"
- board text added: "12V 5V 3V3 GND"
- board text added: "15 14 13 12 11 10 9 8 7 6 5 4 3 2 1 0"
- board text added: "ADC (Load Cells) +0- +1- +2- +3-"
- board text added: "Ematch"
- board text added: "Ext-3V3"
- board text added: "GND 5V S"
- board text added: "Jump for single-ended"
- board text added: "Pressure Transducers 1 2 3"
- board text added: "S 5V G"
- board text added: "SDA SCL 3V3 GND"
- board text added: "Safe-ARM"
- board text added: "Servos"
- board text added: "Sn"
- board text added: "Thermocouples -1+ -2+ -3+ -4+"
- board text added: "[2, 15 V]"
- board text removed: "Thermocouples"
- board text removed: "[3, 15 V]"

Commit message: Edward appeasement
Parts:
- added C32: 100n, Capacitor_SMD:C_0603_1608Metric, F.Cu at (155.8, 126.2)
- added D8: ARM, LED_SMD:LED_0603_1608Metric_Castellated, F.Cu at (164.2, 83.0)
- added J38: Conn_01x02, Connector_PinHeader_2.54mm:PinHeader_1x02_P2.54mm_Vertical, F.Cu at (101.5, 128.0)
- added J39: Conn_01x03, Connector_JST:JST_XH_B3B-XH-A_1x03_P2.50mm_Vertical, F.Cu at (143.7, 111.7)
- added J40: Conn_01x03, Connector_JST:JST_XH_B3B-XH-A_1x03_P2.50mm_Vertical, F.Cu at (149.9, 111.7)
- added R36: 470, Resistor_SMD:R_0603_1608Metric, F.Cu at (162.5, 83.0)
- added R37: 22k, Resistor_SMD:R_0603_1608Metric, F.Cu at (145.1, 120.5)
- added R38: 43k, Resistor_SMD:R_0603_1608Metric, F.Cu at (142.1, 120.5)
- added R39: 22k, Resistor_SMD:R_0603_1608Metric, F.Cu at (151.1, 120.5)
- added R40: 43k, Resistor_SMD:R_0603_1608Metric, F.Cu at (148.1, 120.5)
- D2: footprint Diode_SMD:D_0603_1608Metric_Castellated -> LED_SMD:LED_0603_1608Metric_Castellated
- J16, J17, J18: footprint Connector_JST:JST_XH_B03B-XH-AM_1x03_P2.50mm_Vertical -> Connector_JST:JST_XH_B3B-XH-A_1x03_P2.50mm_Vertical
- moved J18 4.44 mm to (137.6, 111.7)
- moved R34 3.68 mm to (139.1, 120.5)
- moved R35 3.68 mm to (135.9, 120.5)
- moved J17 3.67 mm to (131.3, 111.7)
- moved R32 3.67 mm to (132.2, 120.5)
- moved R33 3.67 mm to (128.9, 120.5)
- moved R31 2.92 mm to (122.8, 120.5)
- moved J16 2.92 mm to (125.2, 111.7)
- moved R30 2.92 mm to (125.9, 120.5)
Connections:
- net Net-(U2-Pad4) renamed /SENSVP
- net Net-(U2-Pad5) renamed /SENSVN
Routing:
- net /SENSVN: track 0.00 -> 73.0 mm, vias 0 -> 2
- net /SENSVP: track 0.00 -> 67.4 mm, vias 0 -> 2
- net +5V: track 151.1 -> 144.3 mm
- net GND: track 105.1 -> 110.9 mm, vias 49 -> 53
- net Net-(J39-Pad3): track 0.00 -> 4.74 mm
- net Net-(J40-Pad3): track 0.00 -> 4.64 mm
- net Net-(D3-Pad2): track 44.1 -> 47.5 mm
- net /PTAP2: track 42.9 -> 40.3 mm
- net /PTAP3: track 50.6 -> 48.2 mm
- net /PTAP1: track 36.3 -> 34.1 mm
- net +3V3: track 41.7 -> 43.6 mm
- net Net-(D8-Pad1): track 0.00 -> 1.71 mm
- net /SCLK: track 76.1 -> 77.6 mm
- net /PYRO: track 77.8 -> 79.1 mm
- net /MISO: track 73.1 -> 74.1 mm
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Other:
- board text added: "10V 5V 3V3 GND"
- board text added: "Pressure Transducers 1 2 3 4 5"
- board text added: "VP VN"
- board text removed: "12V 5V 3V3 GND"
- board text removed: "Pressure Transducers 1 2 3"
