File: ptaps.sch (KiCad schematic (older format))
At the start: 9 parts

Commit message: Release candidate
Parts:
- gave numbers to parts that had none: 9
Changed lines of the file:
@@
 $Descr A4 11693 8268
 encoding utf-8
-Sheet 6 6
+Sheet 6 7
 Title ""
 Date ""
@@
 $EndDescr
 $Comp
-L Connector_Generic:Conn_01x03 J?
+L Connector_Generic:Conn_01x03 J16
 U 1 1 5DD0A0E4
 P 4000 2950
-F 0 "J?" H 4080 2992 50  0000 L CNN
+F 0 "J16" H 4080 2992 50  0000 L CNN
 F 1 "Conn_01x03" H 4080 2901 50  0000 L CNN
 F 2 "Connector_JST:JST_XH_B03B-XH-AM_1x03_P2.50mm_Vertical" H 4000 2950 50  0001 C CNN
@@
 $EndComp
 $Comp
-L power:GND #PWR?
+L power:GND #PWR0112
 U 1 1 5DD0CBEA
 P 3550 3000
-F 0 "#PWR?" H 3550 2750 50  0001 C CNN
+F 0 "#PWR0112" H 3550 2750 50  0001 C CNN
 F 1 "GND" H 3555 2827 50  0000 C CNN
 F 2 "" H 3550 3000 50  0001 C CNN
@@
 $EndComp
 $Comp
-L power:+5V #PWR?
+L power:+5V #PWR0113
 U 1 1 5DD0BC1A
 P 3500 2850
-F 0 "#PWR?" H 3500 2700 50  0001 C CNN
+F 0 "#PWR0113" H 3500 2700 50  0001 C CNN
 F 1 "+5V" H 3515 3023 50  0000 C CNN
 F 2 "" H 3500 2850 50  0001 C CNN
@@
 Centre positive for safety during wire reversals
 $Comp
-L Device:R_Small R?
+L Device:R_Small R30
 U 1 1 5DD12924
 P 3700 3200
-F 0 "R?" H 3759 3246 50  0000 L CNN
+F 0 "R30" H 3759 3246 50  0000 L CNN
 F 1 "22k" H 3759 3155 50  0000 L CNN
 F 2 "Resistor_SMD:R_0603_1608Metric" H 3700 3200 50  0001 C CNN
@@
 	3700 3050 3800 3050
 $Comp
-L Device:R_Small R?
+L Device:R_Small R31
 U 1 1 5DD1309E
 P 3700 3500
-F 0 "R?" H 3759 3546 50  0000 L CNN
+F 0 "R31" H 3759 3546 50  0000 L CNN
 F 1 "43k" H 3759 3455 50  0000 L CNN
 F 2 "Resistor_SMD:R_0603_1608Metric" H 3700 3500 50  0001 C CNN
@@
 $EndComp
 $Comp
-L power:GND #PWR?
+L power:GND #PWR0114
 U 1 1 5DD13E80
 P 3700 3650
-F 0 "#PWR?" H 3700 3400 50  0001 C CNN
+F 0 "#PWR0114" H 3700 3400 50  0001 C CNN
 F 1 "GND" H 3705 3477 50  0000 C CNN
 F 2 "" H 3700 3650 50  0001 C CNN
@@
 PTAP1
 $Comp
-L Connector_Generic:Conn_01x03 J?
+L Connector_Generic:Conn_01x03 J17
 U 1 1 5DD1A9B8
 P 5100 2950
-F 0 "J?" H 5180 2992 50  0000 L CNN
+F 0 "J17" H 5180 2992 50  0000 L CNN
 F 1 "Conn_01x03" H 5180 2901 50  0000 L CNN
 F 2 "Connector_JST:JST_XH_B03B-XH-AM_1x03_P2.50mm_Vertical" H 5100 2950 50  0001 C CNN
@@
 $EndComp
 $Comp
-L power:GND #PWR?
+L power:GND #PWR0115
 U 1 1 5DD1A9C2
 P 4650 3000
-F 0 "#PWR?" H 4650 2750 50  0001 C CNN
+F 0 "#PWR0115" H 4650 2750 50  0001 C CNN
 F 1 "GND" H 4655 2827 50  0000 C CNN
 F 2 "" H 4650 3000 50  0001 C CNN
@@
 $EndComp
 $Comp
-L power:+5V #PWR?
+L power:+5V #PWR0116
 U 1 1 5DD1A9CC
 P 4600 2850
-F 0 "#PWR?" H 4600 2700 50  0001 C CNN
+F 0 "#PWR0116" H 4600 2700 50  0001 C CNN
 F 1 "+5V" H 4615 3023 50  0000 C CNN
 F 2 "" H 4600 2850 50  0001 C CNN
@@
 	4600 2950 4900 2950
 $Comp
-L Device:R_Small R?
+L Device:R_Small R32
 U 1 1 5DD1A9DA
 P 4800 3200
-F 0 "R?" H 4859 3246 50  0000 L CNN
+F 0 "R32" H 4859 3246 50  0000 L CNN
 F 1 "22k" H 4859 3155 50  0000 L CNN
 F 2 "Resistor_SMD:R_0603_1608Metric" H 4800 3200 50  0001 C CNN
@@
 	4800 3050 4900 3050
 $Comp
-L Device:R_Small R?
+L Device:R_Small R33
 U 1 1 5DD1A9E6
 P 4800 3500
-F 0 "R?" H 4859 3546 50  0000 L CNN
+F 0 "R33" H 4859 3546 50  0000 L CNN
 F 1 "43k" H 4859 3455 50  0000 L CNN
 F 2 "Resistor_SMD:R_0603_1608Metric" H 4800 3500 50  0001 C CNN
@@
 $EndComp
 $Comp
-L power:GND #PWR?
+L power:GND #PWR0117
 U 1 1 5DD1A9F0
 P 4800 3650
-F 0 "#PWR?" H 4800 3400 50  0001 C CNN
+F 0 "#PWR0117" H 4800 3400 50  0001 C CNN
 F 1 "GND" H 4805 3477 50  0000 C CNN
 F 2 "" H 4800 3650 50  0001 C CNN
@@
 PTAP2
 $Comp
-L Connector_Generic:Conn_01x03 J?
+L Connector_Generic:Conn_01x03 J18
 U 1 1 5DD242FB
 P 6150 2950
-F 0 "J?" H 6230 2992 50  0000 L CNN
+F 0 "J18" H 6230 2992 50  0000 L CNN
 F 1 "Conn_01x03" H 6230 2901 50  0000 L CNN
 F 2 "Connector_JST:JST_XH_B03B-XH-AM_1x03_P2.50mm_Vertical" H 6150 2950 50  0001 C CNN
@@
 $EndComp
 $Comp
-L power:GND #PWR?
+L power:GND #PWR0118
 U 1 1 5DD24305
 P 5700 3000
-F 0 "#PWR?" H 5700 2750 50  0001 C CNN
+F 0 "#PWR0118" H 5700 2750 50  0001 C CNN
 F 1 "GND" H 5705 2827 50  0000 C CNN
 F 2 "" H 5700 3000 50  0001 C CNN
@@
 $EndComp
 $Comp
-L power:+5V #PWR?
+L power:+5V #PWR0119
 U 1 1 5DD2430F
 P 5650 2850
-F 0 "#PWR?" H 5650 2700 50  0001 C CNN
+F 0 "#PWR0119" H 5650 2700 50  0001 C CNN
 F 1 "+5V" H 5665 3023 50  0000 C CNN
 F 2 "" H 5650 2850 50  0001 C CNN
@@
 	5650 2950 5950 2950
 $Comp
-L Device:R_Small R?
+L Device:R_Small R34
 U 1 1 5DD2431D
 P 5850 3200
-F 0 "R?" H 5909 3246 50  0000 L CNN
+F 0 "R34" H 5909 3246 50  0000 L CNN
 F 1 "22k" H 5909 3155 50  0000 L CNN
 F 2 "Resistor_SMD:R_0603_1608Metric" H 5850 3200 50  0001 C CNN
@@
 	5850 3050 5950 3050
 $Comp
-L Device:R_Small R?
+L Device:R_Small R35
 U 1 1 5DD24329
 P 5850 3500
-F 0 "R?" H 5909 3546 50  0000 L CNN
+F 0 "R35" H 5909 3546 50  0000 L CNN
 F 1 "43k" H 5909 3455 50  0000 L CNN
 F 2 "Resistor_SMD:R_0603_1608Metric" H 5850 3500 50  0001 C CNN
@@
 $EndComp
 $Comp
-L power:GND #PWR?
+L power:GND #PWR0120
 U 1 1 5DD24333
 P 5850 3650
-F 0 "#PWR?" H 5850 3400 50  0001 C CNN
+F 0 "#PWR0120" H 5850 3400 50  0001 C CNN
 F 1 "GND" H 5855 3477 50  0000 C CNN
 F 2 "" H 5850 3650 50  0001 C CNN

Commit message: Edward appeasement
Parts:
- added J39, J40: Conn_01x03, Connector_JST:JST_XH_B3B-XH-A_1x03_P2.50mm_Vertical, symbol Connector_Generic:Conn_01x03
- added R37, R39: 22k, Resistor_SMD:R_0603_1608Metric, symbol Device:R_Small
- added R38, R40: 43k, Resistor_SMD:R_0603_1608Metric, symbol Device:R_Small
- J16, J17, J18: footprint Connector_JST:JST_XH_B03B-XH-AM_1x03_P2.50mm_Vertical -> Connector_JST:JST_XH_B3B-XH-A_1x03_P2.50mm_Vertical
Connections:
- net +5V: now also J39.2 (Pin_2), J40.2 (Pin_2)
- net GND: now also J39.1 (Pin_1), J40.1 (Pin_1), R38.2, R40.2
- new net: J39.3 (Pin_3), R37.1
- new net: J40.3 (Pin_3), R39.1
- new net PTAP4: R37.2, R38.1
- new net PTAP5: R39.2, R40.1
Changed lines of the file:
@@
 F 0 "J16" H 4080 2992 50  0000 L CNN
 F 1 "Conn_01x03" H 4080 2901 50  0000 L CNN
-F 2 "Connector_JST:JST_XH_B03B-XH-AM_1x03_P2.50mm_Vertical" H 4000 2950 50  0001 C CNN
+F 2 "Connector_JST:JST_XH_B3B-XH-A_1x03_P2.50mm_Vertical" H 4000 2950 50  0001 C CNN
 F 3 "~" H 4000 2950 50  0001 C CNN
 	1    4000 2950
@@
 Wire Wire Line
 	3500 2950 3800 2950
-Text Notes 4150 4200 0    50   ~ 0
+Text Notes 4900 4150 0    50   ~ 0
 Centre positive for safety during wire reversals
 $Comp
@@
 F 0 "J17" H 5180 2992 50  0000 L CNN
 F 1 "Conn_01x03" H 5180 2901 50  0000 L CNN
-F 2 "Connector_JST:JST_XH_B03B-XH-AM_1x03_P2.50mm_Vertical" H 5100 2950 50  0001 C CNN
+F 2 "Connector_JST:JST_XH_B3B-XH-A_1x03_P2.50mm_Vertical" H 5100 2950 50  0001 C CNN
 F 3 "~" H 5100 2950 50  0001 C CNN
 	1    5100 2950
@@
 F 0 "J18" H 6230 2992 50  0000 L CNN
 F 1 "Conn_01x03" H 6230 2901 50  0000 L CNN
-F 2 "Connector_JST:JST_XH_B03B-XH-AM_1x03_P2.50mm_Vertical" H 6150 2950 50  0001 C CNN
+F 2 "Connector_JST:JST_XH_B3B-XH-A_1x03_P2.50mm_Vertical" H 6150 2950 50  0001 C CNN
 F 3 "~" H 6150 2950 50  0001 C CNN
 	1    6150 2950
@@
 Text HLabel 5950 3350 2    50   Output ~ 0
 PTAP3
+$Comp
+L Connector_Generic:Conn_01x03 J39
+U 1 1 5E17A0A4
+P 7250 2950
+F 0 "J39" H 7330 2992 50  0000 L CNN
+F 1 "Conn_01x03" H 7330 2901 50  0000 L CNN
+F 2 "Connector_JST:JST_XH_B3B-XH-A_1x03_P2.50mm_Vertical" H 7250 2950 50  0001 C CNN
+F 3 "~" H 7250 2950 50  0001 C CNN
+	1    7250 2950
+	1    0    0    -1
+$EndComp
+$Comp
+L power:GND #PWR0182
+U 1 1 5E17A0AE
+P 6800 3000
+F 0 "#PWR0182" H 6800 2750 50  0001 C CNN
+F 1 "GND" H 6805 2827 50  0000 C CNN
+F 2 "" H 6800 3000 50  0001 C CNN
+F 3 "" H 6800 3000 50  0001 C CNN
+	1    6800 3000
+	1    0    0    -1
+$EndComp
+$Comp
+L power:+5V #PWR0183
+U 1 1 5E17A0B8
+P 6750 2850
+F 0 "#PWR0183" H 6750 2700 50  0001 C CNN
+F 1 "+5V" H 6765 3023 50  0000 C CNN
+F 2 "" H 6750 2850 50  0001 C CNN
+F 3 "" H 6750 2850 50  0001 C CNN
+	1    6750 2850
+	1    0    0    -1
+$EndComp
+Wire Wire Line
+	6800 3000 6800 2850
+Wire Wire Line
+	6800 2850 7050 2850
+Wire Wire Line
+	6750 2850 6750 2950
+Wire Wire Line
+	6750 2950 7050 2950
+$Comp
+L Device:R_Small R37
+U 1 1 5E17A0C6
+P 6950 3200
+F 0 "R37" H 7009 3246 50  0000 L CNN
+F 1 "22k" H 7009 3155 50  0000 L CNN
+F 2 "Resistor_SMD:R_0603_1608Metric" H 6950 3200 50  0001 C CNN
+F 3 "~" H 6950 3200 50  0001 C CNN
+	1    6950 3200
+	1    0    0    -1
+$EndComp
+Wire Wire Line
+	6950 3100 6950 3050
+Wire Wire Line
+	6950 3050 7050 3050
+$Comp
+L Device:R_Small R38
+U 1 1 5E17A0D2
+P 6950 3500
+F 0 "R38" H 7009 3546 50  0000 L CNN
+F 1 "43k" H 7009 3455 50  0000 L CNN
+F 2 "Resistor_SMD:R_0603_1608Metric" H 6950 3500 50  0001 C CNN
+F 3 "~" H 6950 3500 50  0001 C CNN
+	1    6950 3500
+	1    0    0    -1
+$EndComp
+$Comp
+L power:GND #PWR0184
+U 1 1 5E17A0DC
+P 6950 3650
+F 0 "#PWR0184" H 6950 3400 50  0001 C CNN
+F 1 "GND" H 6955 3477 50  0000 C CNN
+F 2 "" H 6950 3650 50  0001 C CNN
+F 3 "" H 6950 3650 50  0001 C CNN
+	1    6950 3650
+	1    0    0    -1
+$EndComp
+Wire Wire Line
+	6950 3650 6950 3600
+Wire Wire Line
+	6950 3400 6950 3350
+Wire Wire Line
+	6950 3350 7050 3350
+Connection ~ 6950 3350
+Wire Wire Line
+	6950 3350 6950 3300
+Text HLabel 7050 3350 2    50   Output ~ 0
+PTAP4
+$Comp
+L Connector_Generic:Conn_01x03 J40
+U 1 1 5E1830C2
+P 8350 2950
+F 0 "J40" H 8430 2992 50  0000 L CNN
+F 1 "Conn_01x03" H 8430 2901 50  0000 L CNN
+F 2 "Connector_JST:JST_XH_B3B-XH-A_1x03_P2.50mm_Vertical" H 8350 2950 50  0001 C CNN
+F 3 "~" H 8350 2950 50  0001 C CNN
+	1    8350 2950
+	1    0    0    -1
+$EndComp
+$Comp
+L power:GND #PWR0185
+U 1 1 5E1830CC
+P 7900 3000
+F 0 "#PWR0185" H 7900 2750 50  0001 C CNN
+F 1 "GND" H 7905 2827 50  0000 C CNN
+F 2 "" H 7900 3000 50  0001 C CNN
+F 3 "" H 7900 3000 50  0001 C CNN
+	1    7900 3000
+	1    0    0    -1
+$EndComp
+$Comp
+L power:+5V #PWR0186
+U 1 1 5E1830D6
+P 7850 2850
+F 0 "#PWR0186" H 7850 2700 50  0001 C CNN
+F 1 "+5V" H 7865 3023 50  0000 C CNN
+F 2 "" H 7850 2850 50  0001 C CNN
+F 3 "" H 7850 2850 50  0001 C CNN
+	1    7850 2850
+	1    0    0    -1
+$EndComp
+Wire Wire Line
+	7900 3000 7900 2850
+Wire Wire Line
+	7900 2850 8150 2850
+Wire Wire Line
+	7850 2850 7850 2950
+Wire Wire Line
+	7850 2950 8150 2950
+$Comp
+L Device:R_Small R39
+U 1 1 5E1830E4
+P 8050 3200
+F 0 "R39" H 8109 3246 50  0000 L CNN
+F 1 "22k" H 8109 3155 50  0000 L CNN
+F 2 "Resistor_SMD:R_0603_1608Metric" H 8050 3200 50  0001 C CNN
+F 3 "~" H 8050 3200 50  0001 C CNN
+	1    8050 3200
+	1    0    0    -1
+$EndComp
+Wire Wire Line
+	8050 3100 8050 3050
+Wire Wire Line
+	8050 3050 8150 3050
+$Comp
+L Device:R_Small R40
+U 1 1 5E1830F0
+P 8050 3500
+F 0 "R40" H 8109 3546 50  0000 L CNN
+F 1 "43k" H 8109 3455 50  0000 L CNN
+F 2 "Resistor_SMD:R_0603_1608Metric" H 8050 3500 50  0001 C CNN
+F 3 "~" H 8050 3500 50  0001 C CNN
+	1    8050 3500
+	1    0    0    -1
+$EndComp
+$Comp
+L power:GND #PWR0187
+U 1 1 5E1830FA
+P 8050 3650
+F 0 "#PWR0187" H 8050 3400 50  0001 C CNN
+F 1 "GND" H 8055 3477 50  0000 C CNN
+F 2 "" H 8050 3650 50  0001 C CNN
+F 3 "" H 8050 3650 50  0001 C CNN
+	1    8050 3650
+	1    0    0    -1
+$EndComp
+Wire Wire Line
+	8050 3650 8050 3600
+Wire Wire Line
+	8050 3400 8050 3350
+Wire Wire Line
+	8050 3350 8150 3350
+Connection ~ 8050 3350
+Wire Wire Line
+	8050 3350 8050 3300
+Text HLabel 8150 3350 2    50   Output ~ 0
+PTAP5
 $EndSCHEMATC
