File: pyro.sch (KiCad schematic (older format))
At the start: 10 parts

Commit message: Not sure if this is gonna overwrite stuff but I try to push this anyway
Parts:
- gave numbers to parts that had none: 10
Changed lines of the file:
@@
 $EndDescr
 $Comp
-L Connector:Screw_Terminal_01x02 J?
+L Connector:Screw_Terminal_01x02 J10
 U 1 1 5DBD0F3F
 P 3550 3100
-F 0 "J?" H 3468 2775 50  0000 C CNN
+F 0 "J10" H 3468 2775 50  0000 C CNN
 F 1 "Screw_Terminal_01x02" H 3468 2866 50  0000 C CNN
 F 2 "TerminalBlock_Phoenix:TerminalBlock_Phoenix_MPT-0,5-2-2.54_1x02_P2.54mm_Horizontal" H 3550 3100 50  0001 C CNN
@@
 $EndComp
 $Comp
-L power:GND #PWR?
+L power:GND #PWR0153
 U 1 1 5DBD3778
 P 3850 3550
-F 0 "#PWR?" H 3850 3300 50  0001 C CNN
+F 0 "#PWR0153" H 3850 3300 50  0001 C CNN
 F 1 "GND" H 3855 3377 50  0000 C CNN
 F 2 "" H 3850 3550 50  0001 C CNN
@@
 	3850 3200 3850 3550
 $Comp
-L Connector:Screw_Terminal_01x02 J?
+L Connector:Screw_Terminal_01x02 J11
 U 1 1 5DBD6464
 P 5100 2700
-F 0 "J?" V 5064 2512 50  0000 R CNN
+F 0 "J11" V 5064 2512 50  0000 R CNN
 F 1 "Screw_Terminal_01x02" V 4973 2512 50  0000 R CNN
 F 2 "TerminalBlock_Phoenix:TerminalBlock_Phoenix_MPT-0,5-2-2.54_1x02_P2.54mm_Horizontal" H 5100 2700 50  0001 C CNN
@@
 $EndComp
 $Comp
-L Device:R R?
+L Device:R R23
 U 1 1 5DBD833E
 P 4650 3350
-F 0 "R?" H 4720 3396 50  0000 L CNN
+F 0 "R23" H 4720 3396 50  0000 L CNN
 F 1 "1k" H 4720 3305 50  0000 L CNN
 F 2 "Resistor_SMD:R_0603_1608Metric" V 4580 3350 50  0001 C CNN
@@
 $EndComp
 $Comp
-L Device:LED D?
+L Device:LED D3
 U 1 1 5DBDDC78
 P 4650 3050
-F 0 "D?" V 4689 2933 50  0000 R CNN
+F 0 "D3" V 4689 2933 50  0000 R CNN
 F 1 "FIRING" V 4598 2933 50  0000 R CNN
 F 2 "LED_SMD:LED_0805_2012Metric" H 4650 3050 50  0001 C CNN
@@
 	4650 2900 5100 2900
 $Comp
-L Simulation_SPICE:DIODE D?
+L Simulation_SPICE:DIODE D4
 U 1 1 5DBDF40B
 P 5200 3300
-F 0 "D?" V 5154 3380 50  0000 L CNN
+F 0 "D4" V 5154 3380 50  0000 L CNN
 F 1 "DIODE" V 5245 3380 50  0000 L CNN
 F 2 "Diode_SMD:D_SMA" H 5200 3300 50  0001 C CNN
@@
 	5200 2900 5200 3050
 $Comp
-L Device:Q_NMOS_GSD Q?
+L Device:Q_NMOS_GSD Q2
 U 1 1 5DBE3E5B
 P 5100 3950
-F 0 "Q?" H 5306 3996 50  0000 L CNN
+F 0 "Q2" H 5306 3996 50  0000 L CNN
 F 1 "PMV20ENR" H 5306 3905 50  0000 L CNN
 F 2 "Package_TO_SOT_SMD:SOT-23" H 5300 4050 50  0001 C CNN
@@
 	5200 4150 5200 4350
 $Comp
-L power:GND #PWR?
+L power:GND #PWR0154
 U 1 1 5DBE510B
 P 5200 4350
-F 0 "#PWR?" H 5200 4100 50  0001 C CNN
+F 0 "#PWR0154" H 5200 4100 50  0001 C CNN
 F 1 "GND" H 5205 4177 50  0000 C CNN
 F 2 "" H 5200 4350 50  0001 C CNN
@@
 	5200 3050 5200 3150
 $Comp
-L Isolator:LTV-817S U?
+L Isolator:LTV-817S U10
 U 1 1 5DBE64FC
 P 6050 3600
-F 0 "U?" H 6050 3925 50  0000 C CNN
+F 0 "U10" H 6050 3925 50  0000 C CNN
 F 1 "LTV-817S" H 6050 3834 50  0000 C CNN
 F 2 "Package_DIP:SMDIP-4_W9.53mm" H 6050 3300 50  0001 C CNN
@@
 	5200 3050 6350 3050
 $Comp
-L Device:R R?
+L Device:R R25
 U 1 1 5DBE9B58
 P 6350 3850
-F 0 "R?" H 6420 3896 50  0000 L CNN
+F 0 "R25" H 6420 3896 50  0000 L CNN
 F 1 "500" H 6420 3805 50  0000 L CNN
 F 2 "Resistor_SMD:R_0603_1608Metric" V 6280 3850 50  0001 C CNN
@@
 	6000 4150 6000 4300
 $Comp
-L power:GND #PWR?
+L power:GND #PWR0155
 U 1 1 5DBEA959
 P 6000 4300
-F 0 "#PWR?" H 6000 4050 50  0001 C CNN
+F 0 "#PWR0155" H 6000 4050 50  0001 C CNN
 F 1 "GND" H 6005 4127 50  0000 C CNN
 F 2 "" H 6000 4300 50  0001 C CNN
@@
 $EndComp
 $Comp
-L power:+3.3V #PWR?
+L power:+3.3V #PWR0156
 U 1 1 5DBEE894
 P 5750 3500
-F 0 "#PWR?" H 5750 3350 50  0001 C CNN
+F 0 "#PWR0156" H 5750 3350 50  0001 C CNN
 F 1 "+3.3V" H 5765 3673 50  0000 C CNN
 F 2 "" H 5750 3500 50  0001 C CNN
@@
 $EndComp
 $Comp
-L Device:R R?
+L Device:R R24
 U 1 1 5DBEF42E
 P 5750 3850
-F 0 "R?" H 5820 3896 50  0000 L CNN
+F 0 "R24" H 5820 3896 50  0000 L CNN
 F 1 "500" H 5820 3805 50  0000 L CNN
 F 2 "Resistor_SMD:R_0603_1608Metric" V 5680 3850 50  0001 C CNN
@@
 	3750 3100 4200 3100
 $Comp
-L Jumper:SolderJumper_3_Open JP?
+L Jumper:SolderJumper_3_Open JP1
 U 1 1 5DB4DA71
 P 4450 2650
-F 0 "JP?" H 4450 2855 50  0000 C CNN
+F 0 "JP1" H 4450 2855 50  0000 C CNN
 F 1 "SolderJumper_3_Open" H 4450 2764 50  0000 C CNN
 F 2 "Jumper:SolderJumper-3_P2.0mm_Open_TrianglePad1.0x1.5mm" H 4450 2650 50  0001 C CNN
@@
 	4200 2650 4200 3100
 $Comp
-L power:+3V3 #PWR?
+L power:+3V3 #PWR0157
 U 1 1 5DB4F735
 P 4950 2500
-F 0 "#PWR?" H 4950 2350 50  0001 C CNN
+F 0 "#PWR0157" H 4950 2350 50  0001 C CNN
 F 1 "+3V3" H 4965 2673 50  0000 C CNN
 F 2 "" H 4950 2500 50  0001 C CNN

Commit message: Fixed conflicts, assigned all footprints.
Parts:
- D4: symbol Simulation_SPICE:DIODE -> Device:D
- renumbered J11 to J10, J10 to J9, R23 to R25, R24 to R26, R25 to R27
Changed lines of the file:
@@
 $Descr A4 11693 8268
 encoding utf-8
-Sheet 6 6
+Sheet 4 5
 Title ""
 Date ""
@@
 $EndDescr
 $Comp
-L Connector:Screw_Terminal_01x02 J10
+L Connector:Screw_Terminal_01x02 J9
 U 1 1 5DBD0F3F
 P 3550 3100
-F 0 "J10" H 3468 2775 50  0000 C CNN
+F 0 "J9" H 3468 2775 50  0000 C CNN
 F 1 "Screw_Terminal_01x02" H 3468 2866 50  0000 C CNN
 F 2 "TerminalBlock_Phoenix:TerminalBlock_Phoenix_MPT-0,5-2-2.54_1x02_P2.54mm_Horizontal" H 3550 3100 50  0001 C CNN
@@
 $EndComp
 $Comp
-L power:GND #PWR0153
+L power:GND #PWR051
 U 1 1 5DBD3778
 P 3850 3550
-F 0 "#PWR0153" H 3850 3300 50  0001 C CNN
+F 0 "#PWR051" H 3850 3300 50  0001 C CNN
 F 1 "GND" H 3855 3377 50  0000 C CNN
 F 2 "" H 3850 3550 50  0001 C CNN
@@
 	3850 3200 3850 3550
 $Comp
-L Connector:Screw_Terminal_01x02 J11
+L Connector:Screw_Terminal_01x02 J10
 U 1 1 5DBD6464
 P 5100 2700
-F 0 "J11" V 5064 2512 50  0000 R CNN
+F 0 "J10" V 5064 2512 50  0000 R CNN
 F 1 "Screw_Terminal_01x02" V 4973 2512 50  0000 R CNN
 F 2 "TerminalBlock_Phoenix:TerminalBlock_Phoenix_MPT-0,5-2-2.54_1x02_P2.54mm_Horizontal" H 5100 2700 50  0001 C CNN
@@
 $EndComp
 $Comp
-L Device:R R23
+L Device:R R25
 U 1 1 5DBD833E
 P 4650 3350
-F 0 "R23" H 4720 3396 50  0000 L CNN
+F 0 "R25" H 4720 3396 50  0000 L CNN
 F 1 "1k" H 4720 3305 50  0000 L CNN
 F 2 "Resistor_SMD:R_0603_1608Metric" V 4580 3350 50  0001 C CNN
@@
 	4650 2900 5100 2900
 $Comp
-L Simulation_SPICE:DIODE D4
+L Device:D D?
 U 1 1 5DBDF40B
 P 5200 3300
+AR Path="/5DBDF40B" Ref="D?"  Part="1"
+AR Path="/5DB4FA2A/5DBDF40B" Ref="D4"  Part="1"
 F 0 "D4" V 5154 3380 50  0000 L CNN
 F 1 "DIODE" V 5245 3380 50  0000 L CNN
@@
 	5200 4150 5200 4350
 $Comp
-L power:GND #PWR0154
+L power:GND #PWR053
 U 1 1 5DBE510B
 P 5200 4350
-F 0 "#PWR0154" H 5200 4100 50  0001 C CNN
+F 0 "#PWR053" H 5200 4100 50  0001 C CNN
 F 1 "GND" H 5205 4177 50  0000 C CNN
 F 2 "" H 5200 4350 50  0001 C CNN
@@
 	5200 3050 6350 3050
 $Comp
-L Device:R R25
+L Device:R R27
 U 1 1 5DBE9B58
 P 6350 3850
-F 0 "R25" H 6420 3896 50  0000 L CNN
+F 0 "R27" H 6420 3896 50  0000 L CNN
 F 1 "500" H 6420 3805 50  0000 L CNN
 F 2 "Resistor_SMD:R_0603_1608Metric" V 6280 3850 50  0001 C CNN
@@
 	6000 4150 6000 4300
 $Comp
-L power:GND #PWR0155
+L power:GND #PWR055
 U 1 1 5DBEA959
 P 6000 4300
-F 0 "#PWR0155" H 6000 4050 50  0001 C CNN
+F 0 "#PWR055" H 6000 4050 50  0001 C CNN
 F 1 "GND" H 6005 4127 50  0000 C CNN
 F 2 "" H 6000 4300 50  0001 C CNN
@@
 $EndComp
 $Comp
-L power:+3.3V #PWR0156
+L power:+3.3V #PWR054
 U 1 1 5DBEE894
 P 5750 3500
-F 0 "#PWR0156" H 5750 3350 50  0001 C CNN
+F 0 "#PWR054" H 5750 3350 50  0001 C CNN
 F 1 "+3.3V" H 5765 3673 50  0000 C CNN
 F 2 "" H 5750 3500 50  0001 C CNN
@@
 $EndComp
 $Comp
-L Device:R R24
+L Device:R R26
 U 1 1 5DBEF42E
 P 5750 3850
-F 0 "R24" H 5820 3896 50  0000 L CNN
+F 0 "R26" H 5820 3896 50  0000 L CNN
 F 1 "500" H 5820 3805 50  0000 L CNN
 F 2 "Resistor_SMD:R_0603_1608Metric" V 5680 3850 50  0001 C CNN
@@
 	4200 2650 4200 3100
 $Comp
-L power:+3V3 #PWR0157
+L power:+3V3 #PWR052
 U 1 1 5DB4F735
 P 4950 2500
-F 0 "#PWR0157" H 4950 2350 50  0001 C CNN
+F 0 "#PWR052" H 4950 2350 50  0001 C CNN
 F 1 "+3V3" H 4965 2673 50  0000 C CNN
 F 2 "" H 4950 2500 50  0001 C CNN

Commit message: Cleaned up layout, added barrel jack for power input
Parts:
- JP1: footprint Jumper:SolderJumper-3_P2.0mm_Open_TrianglePad1.0x1.5mm -> Jumper:SolderJumper-3_P1.3mm_Open_RoundedPad1.0x1.5mm_NumberLabels
Changed lines of the file:
@@
 F 0 "JP1" H 4450 2855 50  0000 C CNN
 F 1 "SolderJumper_3_Open" H 4450 2764 50  0000 C CNN
-F 2 "Jumper:SolderJumper-3_P2.0mm_Open_TrianglePad1.0x1.5mm" H 4450 2650 50  0001 C CNN
+F 2 "Jumper:SolderJumper-3_P1.3mm_Open_RoundedPad1.0x1.5mm_NumberLabels" H 4450 2650 50  0001 C CNN
 F 3 "~" H 4450 2650 50  0001 C CNN
 	1    4450 2650

Commit message: Added 3D models, added ptaps sheet, fixed pyros
Parts:
- removed D4: DIODE, Diode_SMD:D_SMA, symbol Device:D
- added D4: D_Schottky, Diode_SMD:D_SOD-123F, symbol Device:D_Schottky
- added D?: CONTINUITY, LED_SMD:LED_0805_2012Metric, symbol Device:LED
- added R?: 470, Resistor_SMD:R_0603_1608Metric, symbol Device:R
- R25: value 1k -> 470
Connections:
- net +3V3: now also U10.4; no longer U10.1
- net GND: now also R?.2
- net at J10.2 (Pin_2): now also U10.1, D4.2 (A), D?.2 (A); no longer U10.4
- net at Q2.3 (D), R25.2: now also D4.1 (K)
- net at R27.1: now also U10.2; no longer U10.3
- net CONT renamed Cont
- net Cont: now also U10.3; no longer U10.2
- new net: D?.1 (K), R?.1
Other:
- moved on the sheet: R26, R27
Changed lines of the file:
@@
 $Descr A4 11693 8268
 encoding utf-8
-Sheet 4 5
+Sheet 4 6
 Title ""
 Date ""
@@
 P 4650 3350
 F 0 "R25" H 4720 3396 50  0000 L CNN
-F 1 "1k" H 4720 3305 50  0000 L CNN
+F 1 "470" H 4720 3305 50  0000 L CNN
 F 2 "Resistor_SMD:R_0603_1608Metric" V 4580 3350 50  0001 C CNN
 F 3 "~" H 4650 3350 50  0001 C CNN
@@
 Wire Wire Line
 	4650 2900 5100 2900
-$Comp
-L Device:D D?
-U 1 1 5DBDF40B
-P 5200 3300
-AR Path="/5DBDF40B" Ref="D?"  Part="1"
-AR Path="/5DB4FA2A/5DBDF40B" Ref="D4"  Part="1"
-F 0 "D4" V 5154 3380 50  0000 L CNN
-F 1 "DIODE" V 5245 3380 50  0000 L CNN
-F 2 "Diode_SMD:D_SMA" H 5200 3300 50  0001 C CNN
-F 3 "~" H 5200 3300 50  0001 C CNN
-F 4 "Y" H 5200 3300 50  0001 L CNN "Spice_Netlist_Enabled"
-F 5 "V" H 5200 3300 50  0001 L CNN "Spice_Primitive"
-	1    5200 3300
-	0    1    1    0
-$EndComp
-Wire Wire Line
-	5200 3450 5200 3500
+Wire Wire Line
+	5200 3400 5200 3500
 Wire Wire Line
 	4650 3500 5200 3500
@@
 Connection ~ 5200 3050
 Wire Wire Line
-	5200 3050 5200 3150
+	5200 3050 5200 3100
 $Comp
 L Isolator:LTV-817S U10
@@
 F 3 "http://www.us.liteon.com/downloads/LTV-817-827-847.PDF" H 5700 3900 50  0001 C CNN
 	1    6050 3600
-	1    0    0    -1
+	-1   0    0    -1
 $EndComp
 Wire Wire Line
@@
 L Device:R R27
 U 1 1 5DBE9B58
-P 6350 3850
-F 0 "R27" H 6420 3896 50  0000 L CNN
-F 1 "500" H 6420 3805 50  0000 L CNN
-F 2 "Resistor_SMD:R_0603_1608Metric" V 6280 3850 50  0001 C CNN
-F 3 "~" H 6350 3850 50  0001 C CNN
-	1    6350 3850
-	1    0    0    -1
-$EndComp
-Wire Wire Line
-	6350 4000 6350 4150
-Wire Wire Line
-	6350 4150 6000 4150
-Wire Wire Line
-	6000 4150 6000 4300
+P 6350 3950
+F 0 "R27" H 6420 3996 50  0000 L CNN
+F 1 "500" H 6420 3905 50  0000 L CNN
+F 2 "Resistor_SMD:R_0603_1608Metric" V 6280 3950 50  0001 C CNN
+F 3 "~" H 6350 3950 50  0001 C CNN
+	1    6350 3950
+	1    0    0    -1
+$EndComp
+Wire Wire Line
+	6350 4150 6050 4150
+Wire Wire Line
+	6050 4150 6050 4200
 $Comp
 L power:GND #PWR055
 U 1 1 5DBEA959
-P 6000 4300
-F 0 "#PWR055" H 6000 4050 50  0001 C CNN
-F 1 "GND" H 6005 4127 50  0000 C CNN
-F 2 "" H 6000 4300 50  0001 C CNN
-F 3 "" H 6000 4300 50  0001 C CNN
-	1    6000 4300
-	1    0    0    -1
-$EndComp
-$Comp
-L power:+3.3V #PWR054
-U 1 1 5DBEE894
-P 5750 3500
-F 0 "#PWR054" H 5750 3350 50  0001 C CNN
-F 1 "+3.3V" H 5765 3673 50  0000 C CNN
-F 2 "" H 5750 3500 50  0001 C CNN
-F 3 "" H 5750 3500 50  0001 C CNN
-	1    5750 3500
+P 6050 4200
+F 0 "#PWR055" H 6050 3950 50  0001 C CNN
+F 1 "GND" H 6055 4027 50  0000 C CNN
+F 2 "" H 6050 4200 50  0001 C CNN
+F 3 "" H 6050 4200 50  0001 C CNN
+	1    6050 4200
 	1    0    0    -1
 $EndComp
@@
 L Device:R R26
 U 1 1 5DBEF42E
-P 5750 3850
-F 0 "R26" H 5820 3896 50  0000 L CNN
-F 1 "500" H 5820 3805 50  0000 L CNN
-F 2 "Resistor_SMD:R_0603_1608Metric" V 5680 3850 50  0001 C CNN
-F 3 "~" H 5750 3850 50  0001 C CNN
-	1    5750 3850
-	1    0    0    -1
-$EndComp
-Wire Wire Line
-	5750 4000 5750 4150
-Wire Wire Line
-	5750 4150 6000 4150
-Connection ~ 6000 4150
+P 5750 3950
+F 0 "R26" H 5820 3996 50  0000 L CNN
+F 1 "500" H 5820 3905 50  0000 L CNN
+F 2 "Resistor_SMD:R_0603_1608Metric" V 5680 3950 50  0001 C CNN
+F 3 "~" H 5750 3950 50  0001 C CNN
+	1    5750 3950
+	1    0    0    -1
+$EndComp
+Wire Wire Line
+	5750 4150 6050 4150
+Connection ~ 6050 4150
 Text Label 4400 3950 0    50   ~ 0
 Fire
 Wire Wire Line
 	5750 3700 5500 3700
-Connection ~ 5750 3700
 Text Label 5500 3700 0    50   ~ 0
 CONT
@@
 Wire Wire Line
 	4200 2650 4200 3100
-$Comp
-L power:+3V3 #PWR052
-U 1 1 5DB4F735
-P 4950 2500
-F 0 "#PWR052" H 4950 2350 50  0001 C CNN
-F 1 "+3V3" H 4965 2673 50  0000 C CNN
-F 2 "" H 4950 2500 50  0001 C CNN
-F 3 "" H 4950 2500 50  0001 C CNN
-	1    4950 2500
-	1    0    0    -1
-$EndComp
-Wire Wire Line
-	4650 2650 4950 2650
-Wire Wire Line
-	4950 2650 4950 2500
+Wire Wire Line
+	4650 2650 4850 2650
+Wire Wire Line
+	4850 2650 4850 2500
 Text Notes 3100 3000 0    50   ~ 0
 External ematch supply
 Text HLabel 4400 3950 0    50   Input ~ 0
 Fire
+$Comp
+L Device:D_Schottky D?
+U 1 1 5DCE52FA
+P 5200 3250
+AR Path="/5DAD2180/5DCE52FA" Ref="D?"  Part="1"
+AR Path="/5DB4FA2A/5DCE52FA" Ref="D4"  Part="1"
+F 0 "D4" V 5246 3171 50  0000 R CNN
+F 1 "D_Schottky" V 5155 3171 50  0000 R CNN
+F 2 "Diode_SMD:D_SOD-123F" H 5200 3250 50  0001 C CNN
+F 3 "http://www.smc-diodes.com/propdf/DSS12U%20THRU%20DSS125U%20N1873%20REV.A.pdf" H 5200 3250 50  0001 C CNN
+	1    5200 3250
+	0    -1   -1   0
+$EndComp
+Wire Wire Line
+	5750 4100 5750 4150
+Wire Wire Line
+	6350 4100 6350 4150
+Wire Wire Line
+	6350 3800 6350 3700
+Wire Wire Line
+	5750 3800 5750 3700
+Connection ~ 5750 3700
+Text HLabel 5500 3700 0    50   Output ~ 0
+Cont
+$Comp
+L Device:R R?
+U 1 1 5DD2B596
+P 6750 3550
+F 0 "R?" H 6820 3596 50  0000 L CNN
+F 1 "470" H 6820 3505 50  0000 L CNN
+F 2 "Resistor_SMD:R_0603_1608Metric" V 6680 3550 50  0001 C CNN
+F 3 "~" H 6750 3550 50  0001 C CNN
+	1    6750 3550
+	1    0    0    -1
+$EndComp
+$Comp
+L Device:LED D?
+U 1 1 5DD2B5A0
+P 6750 3250
+F 0 "D?" V 6789 3133 50  0000 R CNN
+F 1 "CONTINUITY" V 6698 3133 50  0000 R CNN
+F 2 "LED_SMD:LED_0805_2012Metric" H 6750 3250 50  0001 C CNN
+F 3 "~" H 6750 3250 50  0001 C CNN
+	1    6750 3250
+	0    -1   -1   0
+$EndComp
+Wire Wire Line
+	6350 3050 6750 3050
+Wire Wire Line
+	6750 3050 6750 3100
+Connection ~ 6350 3050
+$Comp
+L power:GND #PWR?
+U 1 1 5DD2EA4C
+P 6750 3750
+F 0 "#PWR?" H 6750 3500 50  0001 C CNN
+F 1 "GND" H 6755 3577 50  0000 C CNN
+F 2 "" H 6750 3750 50  0001 C CNN
+F 3 "" H 6750 3750 50  0001 C CNN
+	1    6750 3750
+	1    0    0    -1
+$EndComp
+Wire Wire Line
+	6750 3750 6750 3700
+$Comp
+L power:+3V3 #PWR052
+U 1 1 5DB4F735
+P 4850 2500
+F 0 "#PWR052" H 4850 2350 50  0001 C CNN
+F 1 "+3V3" H 4865 2673 50  0000 C CNN
+F 2 "" H 4850 2500 50  0001 C CNN
+F 3 "" H 4850 2500 50  0001 C CNN
+	1    4850 2500
+	1    0    0    -1
+$EndComp
+$Comp
+L power:+3V3 #PWR?
+U 1 1 5DD30CD3
+P 5750 3500
+F 0 "#PWR?" H 5750 3350 50  0001 C CNN
+F 1 "+3V3" H 5765 3673 50  0000 C CNN
+F 2 "" H 5750 3500 50  0001 C CNN
+F 3 "" H 5750 3500 50  0001 C CNN
+	1    5750 3500
+	1    0    0    -1
+$EndComp
 $EndSCHEMATC

Commit message: Release candidate
Parts:
- added SW?: SW_DPDT_x2, Button_Switch_THT:SW_CuK_JS202011AQN_DPDT_Angled, symbol Switch:SW_DPDT_x2
- added SW?: SW_DPDT_x2, symbol Switch:SW_DPDT_x2
- D3: footprint LED_SMD:LED_0805_2012Metric -> LED_SMD:LED_0603_1608Metric_Castellated
- D7: renamed from D?; footprint LED_SMD:LED_0805_2012Metric -> LED_SMD:LED_0603_1608Metric_Castellated
- gave numbers to parts that had none: 1
Connections:
- net at D3.2 (A), J10.1 (Pin_1): now also SW?.3 (C), SW?.6 (C); no longer JP1.2 (C)
- new net: JP1.2 (C), SW?.2 (B), SW?.5 (B)
- new net: SW?.1 (A), SW?.4 (A)
Other:
- moved on the sheet: J9, JP1
Changed lines of the file:
@@
 $Descr A4 11693 8268
 encoding utf-8
-Sheet 4 6
+Sheet 4 7
 Title ""
 Date ""
@@
 L Connector:Screw_Terminal_01x02 J9
 U 1 1 5DBD0F3F
-P 3550 3100
-F 0 "J9" H 3468 2775 50  0000 C CNN
-F 1 "Screw_Terminal_01x02" H 3468 2866 50  0000 C CNN
-F 2 "TerminalBlock_Phoenix:TerminalBlock_Phoenix_MPT-0,5-2-2.54_1x02_P2.54mm_Horizontal" H 3550 3100 50  0001 C CNN
-F 3 "~" H 3550 3100 50  0001 C CNN
-	1    3550 3100
+P 2300 1800
+F 0 "J9" H 2218 1475 50  0000 C CNN
+F 1 "Screw_Terminal_01x02" H 2218 1566 50  0000 C CNN
+F 2 "TerminalBlock_Phoenix:TerminalBlock_Phoenix_MPT-0,5-2-2.54_1x02_P2.54mm_Horizontal" H 2300 1800 50  0001 C CNN
+F 3 "~" H 2300 1800 50  0001 C CNN
+	1    2300 1800
 	-1   0    0    -1
 $EndComp
@@
 L power:GND #PWR051
 U 1 1 5DBD3778
-P 3850 3550
-F 0 "#PWR051" H 3850 3300 50  0001 C CNN
-F 1 "GND" H 3855 3377 50  0000 C CNN
-F 2 "" H 3850 3550 50  0001 C CNN
-F 3 "" H 3850 3550 50  0001 C CNN
-	1    3850 3550
-	1    0    0    -1
-$EndComp
-Wire Wire Line
-	3750 3200 3850 3200
-Wire Wire Line
-	3850 3200 3850 3550
+P 2600 2250
+F 0 "#PWR051" H 2600 2000 50  0001 C CNN
+F 1 "GND" H 2605 2077 50  0000 C CNN
+F 2 "" H 2600 2250 50  0001 C CNN
+F 3 "" H 2600 2250 50  0001 C CNN
+	1    2600 2250
+	1    0    0    -1
+$EndComp
+Wire Wire Line
+	2500 1900 2600 1900
+Wire Wire Line
+	2600 1900 2600 2250
 $Comp
 L Connector:Screw_Terminal_01x02 J10
@@
 F 0 "D3" V 4689 2933 50  0000 R CNN
 F 1 "FIRING" V 4598 2933 50  0000 R CNN
-F 2 "LED_SMD:LED_0805_2012Metric" H 4650 3050 50  0001 C CNN
+F 2 "LED_SMD:LED_0603_1608Metric_Castellated" H 4650 3050 50  0001 C CNN
 F 3 "~" H 4650 3050 50  0001 C CNN
 	1    4650 3050
@@
 CONT
 Wire Wire Line
-	3750 3100 4200 3100
+	2500 1800 2950 1800
 $Comp
 L Jumper:SolderJumper_3_Open JP1
 U 1 1 5DB4DA71
-P 4450 2650
-F 0 "JP1" H 4450 2855 50  0000 C CNN
-F 1 "SolderJumper_3_Open" H 4450 2764 50  0000 C CNN
-F 2 "Jumper:SolderJumper-3_P1.3mm_Open_RoundedPad1.0x1.5mm_NumberLabels" H 4450 2650 50  0001 C CNN
-F 3 "~" H 4450 2650 50  0001 C CNN
-	1    4450 2650
-	1    0    0    -1
-$EndComp
-Wire Wire Line
-	4450 2800 4450 2900
-Wire Wire Line
-	4450 2900 4650 2900
+P 3200 2050
+F 0 "JP1" H 3200 2255 50  0000 C CNN
+F 1 "SolderJumper_3_Open" H 3200 2164 50  0000 C CNN
+F 2 "Jumper:SolderJumper-3_P1.3mm_Open_RoundedPad1.0x1.5mm_NumberLabels" H 3200 2050 50  0001 C CNN
+F 3 "~" H 3200 2050 50  0001 C CNN
+	1    3200 2050
+	1    0    0    -1
+$EndComp
 Connection ~ 4650 2900
 Wire Wire Line
-	4200 2650 4250 2650
-Wire Wire Line
-	4200 2650 4200 3100
-Wire Wire Line
-	4650 2650 4850 2650
-Wire Wire Line
-	4850 2650 4850 2500
-Text Notes 3100 3000 0    50   ~ 0
+	2950 2050 3000 2050
+Wire Wire Line
+	2950 2050 2950 1800
+Wire Wire Line
+	3400 2050 3600 2050
+Wire Wire Line
+	3600 2050 3600 1900
+Text Notes 1850 1700 0    50   ~ 0
 External ematch supply
 Text HLabel 4400 3950 0    50   Input ~ 0
@@
 Cont
 $Comp
-L Device:R R?
+L Device:R R29
 U 1 1 5DD2B596
 P 6750 3550
-F 0 "R?" H 6820 3596 50  0000 L CNN
+F 0 "R29" H 6820 3596 50  0000 L CNN
 F 1 "470" H 6820 3505 50  0000 L CNN
 F 2 "Resistor_SMD:R_0603_1608Metric" V 6680 3550 50  0001 C CNN
@@
 $EndComp
 $Comp
-L Device:LED D?
+L Device:LED D7
 U 1 1 5DD2B5A0
 P 6750 3250
-F 0 "D?" V 6789 3133 50  0000 R CNN
+F 0 "D7" V 6789 3133 50  0000 R CNN
 F 1 "CONTINUITY" V 6698 3133 50  0000 R CNN
-F 2 "LED_SMD:LED_0805_2012Metric" H 6750 3250 50  0001 C CNN
+F 2 "LED_SMD:LED_0603_1608Metric_Castellated" H 6750 3250 50  0001 C CNN
 F 3 "~" H 6750 3250 50  0001 C CNN
 	1    6750 3250
@@
 Connection ~ 6350 3050
 $Comp
-L power:GND #PWR?
+L power:GND #PWR0110
 U 1 1 5DD2EA4C
 P 6750 3750
-F 0 "#PWR?" H 6750 3500 50  0001 C CNN
+F 0 "#PWR0110" H 6750 3500 50  0001 C CNN
 F 1 "GND" H 6755 3577 50  0000 C CNN
 F 2 "" H 6750 3750 50  0001 C CNN
@@
 L power:+3V3 #PWR052
 U 1 1 5DB4F735
-P 4850 2500
-F 0 "#PWR052" H 4850 2350 50  0001 C CNN
-F 1 "+3V3" H 4865 2673 50  0000 C CNN
-F 2 "" H 4850 2500 50  0001 C CNN
-F 3 "" H 4850 2500 50  0001 C CNN
-	1    4850 2500
-	1    0    0    -1
-$EndComp
-$Comp
-L power:+3V3 #PWR?
+P 3600 1900
+F 0 "#PWR052" H 3600 1750 50  0001 C CNN
+F 1 "+3V3" H 3615 2073 50  0000 C CNN
+F 2 "" H 3600 1900 50  0001 C CNN
+F 3 "" H 3600 1900 50  0001 C CNN
+	1    3600 1900
+	1    0    0    -1
+$EndComp
+$Comp
+L power:+3V3 #PWR0111
 U 1 1 5DD30CD3
 P 5750 3500
-F 0 "#PWR?" H 5750 3350 50  0001 C CNN
+F 0 "#PWR0111" H 5750 3350 50  0001 C CNN
 F 1 "+3V3" H 5765 3673 50  0000 C CNN
 F 2 "" H 5750 3500 50  0001 C CNN
@@
 	1    0    0    -1
 $EndComp
+$Comp
+L Switch:SW_DPDT_x2 SW?
+U 1 1 5E12E318
+P 3800 2550
+F 0 "SW?" H 3800 2835 50  0000 C CNN
+F 1 "SW_DPDT_x2" H 3800 2744 50  0000 C CNN
+F 2 "Button_Switch_THT:SW_CuK_JS202011AQN_DPDT_Angled" H 3800 2550 50  0001 C CNN
+F 3 "~" H 3800 2550 50  0001 C CNN
+	1    3800 2550
+	1    0    0    -1
+$EndComp
+$Comp
+L Switch:SW_DPDT_x2 SW?
+U 2 1 5E133738
+P 3750 3050
+F 0 "SW?" H 3750 3335 50  0000 C CNN
+F 1 "SW_DPDT_x2" H 3750 3244 50  0000 C CNN
+F 2 "" H 3750 3050 50  0001 C CNN
+F 3 "~" H 3750 3050 50  0001 C CNN
+	2    3750 3050
+	1    0    0    -1
+$EndComp
+Wire Wire Line
+	3950 2950 4100 2950
+Wire Wire Line
+	4100 2950 4100 2450
+Wire Wire Line
+	4100 2450 4000 2450
+Wire Wire Line
+	4000 2650 4200 2650
+Wire Wire Line
+	4200 2650 4200 2900
+Wire Wire Line
+	4200 3150 3950 3150
+Wire Wire Line
+	3550 3050 3450 3050
+Wire Wire Line
+	3450 3050 3450 2800
+Wire Wire Line
+	3450 2550 3600 2550
+Wire Wire Line
+	4200 2900 4650 2900
+Connection ~ 4200 2900
+Wire Wire Line
+	4200 2900 4200 3150
+Wire Wire Line
+	3450 2800 3200 2800
+Wire Wire Line
+	3200 2200 3200 2800
+Connection ~ 3450 2800
+Wire Wire Line
+	3450 2800 3450 2550
 $EndSCHEMATC
